Commit message: Update arm coordination

File: urdf/larm.urdf.xacro (robot description, xacro)
@@ -57,5 +57,5 @@
     </joint>
     <joint name="${prefix}_ely_joint" type="revolute">
-      <origin xyz="0 0.02472 -0.05011" rpy="0 0 0"/>
+      <origin xyz="0 0.05587567 0" rpy="0 0 0"/>
       <axis xyz="0 1 0"/>
       <limit lower="${-pi/2.0}" upper="${pi/2.0}" effort="0" velocity="0"/>
@@ -64,5 +64,5 @@
     </joint>
     <joint name="${prefix}_elx_joint" type="revolute">
-      <origin xyz="0 0.01329 -0.02744" rpy="0 0 0"/>
+      <origin xyz="0 0.030488976696505 0" rpy="0 0 0"/>
       <axis xyz="1 0 0"/>
       <limit lower="${-pi/2.0}" upper="${pi/2.0}" effort="0" velocity="0"/>
@@ -71,5 +71,5 @@
     </joint>
     <joint name="${prefix}_wry_joint" type="revolute">
-      <origin xyz="-0.01002 0.01922 -0.04356" rpy="0 0 0"/>
+      <origin xyz="0.01002 0.047611784255581 0" rpy="0 0 0"/>
       <axis xyz="0 1 0"/>
       <limit lower="${-pi/2.0}" upper="${pi/2.0}" effort="0" velocity="0"/>

File: urdf/rarm.urdf.xacro (robot description, xacro)
@@ -57,5 +57,5 @@
     </joint>
     <joint name="${prefix}_ely_joint" type="revolute">
-      <origin xyz="0 -0.02472 -0.05011" rpy="0 0 0"/>
+      <origin xyz="0 -0.05587567 0" rpy="0 0 0"/>
       <axis xyz="0 1 0"/>
       <limit lower="${-pi/2.0}" upper="${pi/2.0}" effort="0" velocity="0"/>
@@ -64,5 +64,5 @@
     </joint>
     <joint name="${prefix}_elx_joint" type="revolute">
-      <origin xyz="0 -0.01329 -0.02744" rpy="0 0 0"/>
+      <origin xyz="0 -0.030488976696505 0" rpy="0 0 0"/>
       <axis xyz="1 0 0"/>
       <limit lower="${-pi/2.0}" upper="${pi/2.0}" effort="0" velocity="0"/>
@@ -71,5 +71,5 @@
     </joint>
     <joint name="${prefix}_wry_joint" type="revolute">
-      <origin xyz="-0.01002 -0.01922 -0.04356" rpy="0 0 0"/>
+      <origin xyz="0.01002 -0.047611784255581 0" rpy="0 0 0"/>
       <axis xyz="0 1 0"/>
       <limit lower="${-pi/2.0}" upper="${pi/2.0}" effort="0" velocity="0"/>
