Commit message: Fix joint names

File: urdf/body.urdf.xacro (robot description, xacro)
@@ -16,4 +16,11 @@
       </visual>
     </link>
+    <link name="head_dummy">
+      <visual>
+        <geometry>
+          <box size="0.01 0.01 0.01" />
+        </geometry>
+      </visual>
+    </link>
     <link name="head">
       <visual>
@@ -28,5 +35,5 @@
       <child link="body"/>
     </joint>
-    <joint name="head_pitch_joint" type="revolute">
+    <joint name="head_ny_joint" type="revolute">
       <origin xyz="-0.0319 0 0.1088" rpy="0 0 0"/>
       <axis xyz="0 1 0"/>
@@ -35,9 +42,16 @@
       <child link="neck"/>
     </joint>
-    <joint name="head_roll_joint" type="revolute">
-      <origin xyz="0 0 0.0362" rpy="0 0 0"/>
+    <joint name="head_nz_joint" type="revolute">
+      <origin xyz="0 0 0" rpy="0 0 0"/>
       <axis xyz="0 0 1"/>
       <limit lower="${-pi/2.0}" upper="${pi/2.0}" effort="0" velocity="0"/>
       <parent link="neck"/>
+      <child link="head_dummy"/>
+    </joint>
+    <joint name="head_nx_joint" type="revolute">
+      <origin xyz="0 0 0.0362" rpy="0 0 0"/>
+      <axis xyz="1 0 0"/>
+      <limit lower="${-pi/2.0}" upper="${pi/2.0}" effort="0" velocity="0"/>
+      <parent link="head_dummy"/>
       <child link="head"/>
     </joint>

File: urdf/larm.urdf.xacro (robot description, xacro)
@@ -42,5 +42,5 @@
       </visual>
     </link>
-    <joint name="${prefix}_1y_joint" type="revolute">
+    <joint name="${prefix}_shy_joint" type="revolute">
       <origin xyz="-0.01726 0.03829 0.097" rpy="0 0 0"/>
       <axis xyz="0 1 0"/>
@@ -49,5 +49,5 @@
       <child link="${prefix}_1y"/>
     </joint>
-    <joint name="${prefix}_1x_joint" type="revolute">
+    <joint name="${prefix}_shx_joint" type="revolute">
       <origin xyz="0 0.01925 0" rpy="0 0 0"/>
       <axis xyz="1 0 0"/>
@@ -56,12 +56,12 @@
       <child link="${prefix}_1x"/>
     </joint>
-    <joint name="${prefix}_2z_joint" type="revolute">
+    <joint name="${prefix}_ely_joint" type="revolute">
       <origin xyz="0 0.02472 -0.05011" rpy="0 0 0"/>
-      <axis xyz="0 0 1"/>
+      <axis xyz="0 1 0"/>
       <limit lower="${-pi/2.0}" upper="${pi/2.0}" effort="0" velocity="0"/>
       <parent link="${prefix}_1x"/>
       <child link="${prefix}_2z"/>
     </joint>
-    <joint name="${prefix}_2x_joint" type="revolute">
+    <joint name="${prefix}_elx_joint" type="revolute">
       <origin xyz="0 0.01329 -0.02744" rpy="0 0 0"/>
       <axis xyz="1 0 0"/>
@@ -70,7 +70,7 @@
       <child link="${prefix}_2x"/>
     </joint>
-    <joint name="${prefix}_hand_joint" type="revolute">
+    <joint name="${prefix}_wry_joint" type="revolute">
       <origin xyz="-0.01002 0.01922 -0.04356" rpy="0 0 0"/>
-      <axis xyz="0 0 1"/>
+      <axis xyz="0 1 0"/>
       <limit lower="${-pi/2.0}" upper="${pi/2.0}" effort="0" velocity="0"/>
       <parent link="${prefix}_2x"/>

File: urdf/lleg.urdf.xacro (robot description, xacro)
@@ -34,5 +34,5 @@
       </visual>
     </link>
-    <link name="${prefix}_3y">
+    <link name="${prefix}_dummy">
       <visual>
         <origin rpy="0 0 0" xyz="0 0 0"/>
@@ -50,5 +50,5 @@
       </visual>
     </link>
-    <joint name="${prefix}_1z_joint" type="revolute">
+    <joint name="${prefix}_hpz_joint" type="revolute">
       <origin xyz="0 0.0217 0.01505" rpy="0 0 0"/>
       <axis xyz="0 0 1"/>
@@ -57,19 +57,19 @@
       <child link="${prefix}_1z"/>
     </joint>
-    <joint name="${prefix}_1y_joint" type="revolute">
+    <joint name="${prefix}_hpx_joint" type="revolute">
       <origin xyz="0 0 -0.05407" rpy="0 0 0"/>
-      <axis xyz="0 1 0"/>
+      <axis xyz="1 0 0"/>
       <limit lower="${-pi/2.0}" upper="${pi/2.0}" effort="0" velocity="0"/>
       <parent link="${prefix}_1z"/>
       <child link="${prefix}_1y"/>
     </joint>
-    <joint name="${prefix}_1x_joint" type="revolute">
+    <joint name="${prefix}_hpy_joint" type="revolute">
       <origin xyz="0 0.01021 -0.03829" rpy="0 0 0"/>
-      <axis xyz="1 0 0"/>
+      <axis xyz="0 1 0"/>
       <limit lower="${-pi/2.0}" upper="${pi/2.0}" effort="0" velocity="0"/>
       <parent link="${prefix}_1y"/>
       <child link="${prefix}_1x"/>
     </joint>
-    <joint name="${prefix}_2y_joint" type="revolute">
+    <joint name="${prefix}_kny_joint" type="revolute">
       <origin xyz="0 0 -0.06827" rpy="0 0 0"/>
       <axis xyz="0 1 0"/>
@@ -78,16 +78,15 @@
       <child link="${prefix}_2y"/>
     </joint>
-    <!-- MUST implement leg 3y to model  -->
-    <joint name="${prefix}_3y_joint" type="fixed">
+    <joint name="${prefix}_aky_joint" type="revolute">
       <axis xyz="0 1 0"/>
       <limit lower="${-pi/2.0}" upper="${pi/2.0}" effort="0" velocity="0"/>
       <parent link="${prefix}_2y"/>
-      <child link="${prefix}_3y"/>
+      <child link="${prefix}_dummy"/>
     </joint>
-    <joint name="${prefix}_3x_joint" type="revolute">
+    <joint name="${prefix}_akx_joint" type="revolute">
       <origin xyz="0 0 -0.06749" rpy="0 0 0"/>
       <axis xyz="1 0 0"/>
       <limit lower="${-pi/2.0}" upper="${pi/2.0}" effort="0" velocity="0"/>
-      <parent link="${prefix}_3y"/>
+      <parent link="${prefix}_dummy"/>
       <child link="${prefix}_foot"/>
     </joint>

File: urdf/rarm.urdf.xacro (robot description, xacro)
@@ -42,5 +42,5 @@
       </visual>
     </link>
-    <joint name="${prefix}_1y_joint" type="revolute">
+    <joint name="${prefix}_shy_joint" type="revolute">
       <origin xyz="-0.01726 -0.03829 0.097" rpy="0 0 0"/>
       <axis xyz="0 1 0"/>
@@ -49,12 +49,12 @@
       <child link="${prefix}_1y"/>
     </joint>
-    <joint name="${prefix}_1x_joint" type="revolute">
+    <joint name="${prefix}_shx_joint" type="revolute">
       <origin xyz="0 -0.01925 0" rpy="0 0 0"/>
-      <axis xyz="0 1 0"/>
+      <axis xyz="1 0 0"/>
       <limit lower="${-pi/2.0}" upper="${pi/2.0}" effort="0" velocity="0"/>
       <parent link="${prefix}_1y"/>
       <child link="${prefix}_1x"/>
     </joint>
-    <joint name="${prefix}_2z_joint" type="revolute">
+    <joint name="${prefix}_ely_joint" type="revolute">
       <origin xyz="0 -0.02472 -0.05011" rpy="0 0 0"/>
       <axis xyz="0 1 0"/>
@@ -63,12 +63,12 @@
       <child link="${prefix}_2z"/>
     </joint>
-    <joint name="${prefix}_2x_joint" type="revolute">
+    <joint name="${prefix}_elx_joint" type="revolute">
       <origin xyz="0 -0.01329 -0.02744" rpy="0 0 0"/>
-      <axis xyz="0 1 0"/>
+      <axis xyz="1 0 0"/>
       <limit lower="${-pi/2.0}" upper="${pi/2.0}" effort="0" velocity="0"/>
       <parent link="${prefix}_2z"/>
       <child link="${prefix}_2x"/>
     </joint>
-    <joint name="${prefix}_hand_joint" type="revolute">
+    <joint name="${prefix}_wry_joint" type="revolute">
       <origin xyz="-0.01002 -0.01922 -0.04356" rpy="0 0 0"/>
       <axis xyz="0 1 0"/>

File: urdf/rleg.urdf.xacro (robot description, xacro)
@@ -34,5 +34,5 @@
       </visual>
     </link>
-    <link name="${prefix}_3y">
+    <link name="${prefix}_dummy">
       <visual>
         <origin rpy="0 0 0" xyz="0 0 0"/>
@@ -50,5 +50,5 @@
       </visual>
     </link>
-    <joint name="${prefix}_1z_joint" type="revolute">
+    <joint name="${prefix}_hpz_joint" type="revolute">
       <origin xyz="0 -0.0217 0.01505" rpy="0 0 0"/>
       <axis xyz="0 0 1"/>
@@ -57,19 +57,19 @@
       <child link="${prefix}_1z"/>
     </joint>
-    <joint name="${prefix}_1y_joint" type="revolute">
+    <joint name="${prefix}_hpx_joint" type="revolute">
       <origin xyz="0 0 -0.05407" rpy="0 0 0"/>
-      <axis xyz="0 1 0"/>
+      <axis xyz="1 0 0"/>
       <limit lower="${-pi/2.0}" upper="${pi/2.0}" effort="0" velocity="0"/>
       <parent link="${prefix}_1z"/>
       <child link="${prefix}_1y"/>
     </joint>
-    <joint name="${prefix}_1x_joint" type="revolute">
+    <joint name="${prefix}_hpy_joint" type="revolute">
       <origin xyz="0 -0.01021 -0.03829" rpy="0 0 0"/>
-      <axis xyz="1 0 0"/>
+      <axis xyz="0 1 0"/>
       <limit lower="${-pi/2.0}" upper="${pi/2.0}" effort="0" velocity="0"/>
       <parent link="${prefix}_1y"/>
       <child link="${prefix}_1x"/>
     </joint>
-    <joint name="${prefix}_2y_joint" type="revolute">
+    <joint name="${prefix}_kny_joint" type="revolute">
       <origin xyz="0 0 -0.06827" rpy="0 0 0"/>
       <axis xyz="0 1 0"/>
@@ -78,16 +78,15 @@
       <child link="${prefix}_2y"/>
     </joint>
-    <!-- MUST implement leg 3y to model  -->
-    <joint name="${prefix}_3y_joint" type="fixed">
+    <joint name="${prefix}_aky_joint" type="revolute">
       <axis xyz="0 1 0"/>
       <limit lower="${-pi/2.0}" upper="${pi/2.0}" effort="0" velocity="0"/>
       <parent link="${prefix}_2y"/>
-      <child link="${prefix}_3y"/>
+      <child link="${prefix}_dummy"/>
     </joint>
-    <joint name="${prefix}_3x_joint" type="revolute">
+    <joint name="${prefix}_akx_joint" type="revolute">
       <origin xyz="0 0 -0.06749" rpy="0 0 0"/>
       <axis xyz="1 0 0"/>
       <limit lower="${-pi/2.0}" upper="${pi/2.0}" effort="0" velocity="0"/>
-      <parent link="${prefix}_3y"/>
+      <parent link="${prefix}_dummy"/>
       <child link="${prefix}_foot"/>
     </joint>

Commit message: Add body joint limit

File: urdf/body.urdf.xacro (robot description, xacro)
@@ -53,5 +53,5 @@
       <origin xyz="-0.0319 0 0.1088" rpy="0 0 0"/>
       <axis xyz="0 1 0"/>
-      <limit lower="${-pi/2.0}" upper="${pi/2.0}" effort="0" velocity="0"/>
+      <limit lower="${-10.125/180.0 * pi}" upper="${23.625/180.0 * pi}" effort="0" velocity="0"/>
       <parent link="body"/>
       <child link="neck"/>
@@ -60,5 +60,5 @@
       <origin xyz="0 0 0" rpy="0 0 0"/>
       <axis xyz="0 0 1"/>
-      <limit lower="${-pi/2.0}" upper="${pi/2.0}" effort="0" velocity="0"/>
+      <limit lower="${-47.25/180.0 * pi}" upper="${47.25/180.0 * pi}" effort="0" velocity="0"/>
       <parent link="neck"/>
       <child link="head_dummy"/>
@@ -67,5 +67,5 @@
       <origin xyz="0 0 0.0362" rpy="0 0 0"/>
       <axis xyz="1 0 0"/>
-      <limit lower="${-pi/2.0}" upper="${pi/2.0}" effort="0" velocity="0"/>
+      <limit lower="${-21.9375/180.0 * pi}" upper="${28.6875/180.0 * pi}" effort="0" velocity="0"/>
       <parent link="head_dummy"/>
       <child link="head"/>
