Commit message: premaidai_description: fix ankle origin in urdf/leg.urdf.xacro

File: urdf/leg.urdf.xacro (robot description, xacro)
@@ -109,4 +109,5 @@
     </joint>
     <joint name="${prefix}_aky_joint" type="revolute">
+      <origin xyz="0 0 -0.06749" rpy="0 0 0"/>
       <axis xyz="0 1 0"/>
       <limit lower="${-pi/2.0}" upper="${pi/2.0}" effort="0" velocity="0"/>
@@ -115,5 +116,4 @@
     </joint>
     <joint name="${prefix}_akx_joint" type="revolute">
-      <origin xyz="0 0 -0.06749" rpy="0 0 0"/>
       <axis xyz="1 0 0"/>
       <limit lower="${-pi/2.0}" upper="${pi/2.0}" effort="0" velocity="0"/>

Commit message: Add leg joint limits

File: urdf/leg.urdf.xacro (robot description, xacro)
@@ -95,5 +95,5 @@
       <xacro:insert_block name="origin" />
       <axis xyz="0 0 1"/>
-      <limit lower="${-pi/2.0}" upper="${pi/2.0}" effort="0" velocity="0"/>
+      <limit lower="${-81.0/180.0 * pi}" upper="${102.43/180.0 * pi}" effort="0" velocity="0"/>
       <parent link="${parent}"/>
       <child link="${prefix}_hip_joint"/>
@@ -102,5 +102,10 @@
       <origin xyz="0 ${sign*-0.0021} -0.028" rpy="0 0 0"/>
       <axis xyz="1 0 0"/>
-      <limit lower="${-pi/2.0}" upper="${pi/2.0}" effort="0" velocity="0"/>
+      <xacro:if value="${side=='right'}">
+        <limit lower="${-25.35/180.0 * pi}" upper="${22.713/180.0 * pi}" effort="0" velocity="0"/>
+      </xacro:if>
+      <xacro:if value="${side=='left'}">
+        <limit lower="${-22.713/180.0 * pi}" upper="${25.35/180.0 * pi}" effort="0" velocity="0"/>
+      </xacro:if>
       <parent link="${prefix}_hip_joint"/>
       <child link="${prefix}_uleg_root"/>
@@ -109,5 +114,5 @@
       <origin xyz="0 ${sign*0.0128525} -0.034358" rpy="0 0 0"/>
       <axis xyz="0 1 0"/>
-      <limit lower="${-pi/2.0}" upper="${pi/2.0}" effort="0" velocity="0"/>
+      <limit lower="${-91.60/180.0 * pi}" upper="${90.213/180.0 * pi}" effort="0" velocity="0"/>
       <parent link="${prefix}_uleg_root"/>
       <child link="${prefix}_uleg"/>
@@ -116,5 +121,5 @@
       <origin xyz="0 0 -0.0652" rpy="0 0 0"/>
       <axis xyz="0 1 0"/>
-      <limit lower="${-pi/2.0}" upper="${pi/2.0}" effort="0" velocity="0"/>
+      <limit lower="${-2.0925/180.0 * pi}" upper="${119.64/180.0 * pi}" effort="0" velocity="0"/>
       <parent link="${prefix}_uleg"/>
       <child link="${prefix}_lleg"/>
@@ -123,5 +128,5 @@
       <origin xyz="0 0 -0.065" rpy="0 0 0"/>
       <axis xyz="0 1 0"/>
-      <limit lower="${-pi/2.0}" upper="${pi/2.0}" effort="0" velocity="0"/>
+      <limit lower="${-61.3575/180.0 * pi}" upper="${24.3/180.0 * pi}" effort="0" velocity="0"/>
       <parent link="${prefix}_lleg"/>
       <child link="${prefix}_ankle"/>
@@ -130,5 +135,10 @@
       <origin xyz="0 0 -0.040677" rpy="0 0 0"/>
       <axis xyz="1 0 0"/>
-      <limit lower="${-pi/2.0}" upper="${pi/2.0}" effort="0" velocity="0"/>
+      <xacro:if value="${side=='right'}">
+        <limit lower="${-38.23875/180.0 * pi}" upper="${37.29375/180.0 * pi}" effort="0" velocity="0"/>
+      </xacro:if>
+      <xacro:if value="${side=='left'}">
+        <limit lower="${-37.29375/180.0 * pi}" upper="${38.23875/180.0 * pi}" effort="0" velocity="0"/>
+      </xacro:if>
       <parent link="${prefix}_ankle"/>
       <child link="${prefix}_foot"/>
