Commit message: Add collision to model

File: urdf/arm.urdf.xacro (robot description, xacro)
@@ -9,4 +9,10 @@
         </geometry>
       </visual>
+      <collision>
+        <origin rpy="0 0 0" xyz="0 0 0"/>
+        <geometry>
+          <mesh filename="package://premaidai_description/meshes/${prefix}_uarm_joint.dae"/>
+        </geometry>
+      </collision>
     </link>
     <link name="${prefix}_uarm">
@@ -17,4 +23,10 @@
         </geometry>
       </visual>
+      <collision>
+        <origin rpy="0 0 0" xyz="0 0 0"/>
+        <geometry>
+          <mesh filename="package://premaidai_description/meshes/${prefix}_uarm.dae"/>
+        </geometry>
+      </collision>
     </link>
     <link name="${prefix}_larm_joint">
@@ -25,4 +37,10 @@
         </geometry>
       </visual>
+      <collision>
+        <origin rpy="0 0 0" xyz="0 0 0"/>
+        <geometry>
+          <mesh filename="package://premaidai_description/meshes/${prefix}_larm_joint.dae"/>
+        </geometry>
+      </collision>
     </link>
     <link name="${prefix}_larm">
@@ -33,4 +51,10 @@
         </geometry>
       </visual>
+      <collision>
+        <origin rpy="0 0 0" xyz="0 0 0"/>
+        <geometry>
+          <mesh filename="package://premaidai_description/meshes/${prefix}_larm.dae"/>
+        </geometry>
+      </collision>
     </link>
     <link name="${prefix}_hand">
@@ -41,4 +65,10 @@
         </geometry>
       </visual>
+      <collision>
+        <origin rpy="0 0 0" xyz="0 0 0"/>
+        <geometry>
+          <mesh filename="package://premaidai_description/meshes/${prefix}_hand.dae"/>
+        </geometry>
+      </collision>
     </link>
     <joint name="${prefix}_shy_joint" type="revolute">

File: urdf/body.urdf.xacro (robot description, xacro)
@@ -8,4 +8,9 @@
         </geometry>
       </visual>
+      <collision>
+        <geometry>
+            <mesh filename="package://premaidai_description/meshes/body.dae"/>
+        </geometry>
+      </collision>
     </link>
     <link name="neck">
@@ -15,4 +20,9 @@
         </geometry>
       </visual>
+      <collision>
+        <geometry>
+            <mesh filename="package://premaidai_description/meshes/neck.dae"/>
+        </geometry>
+      </collision>
     </link>
     <link name="head_dummy">
@@ -29,4 +39,9 @@
         </geometry>
       </visual>
+      <collision>
+        <geometry>
+            <mesh filename="package://premaidai_description/meshes/head.dae"/>
+        </geometry>
+      </collision>
     </link>
     <joint name="body_to_base_link" type="fixed">

File: urdf/leg.urdf.xacro (robot description, xacro)
@@ -9,4 +9,10 @@
         </geometry>
       </visual>
+      <collision>
+        <origin rpy="0 0 0" xyz="0 0 0"/>
+        <geometry>
+          <mesh filename="package://premaidai_description/meshes/${prefix}_hip_joint.dae"/>
+        </geometry>
+      </collision>
     </link>
     <link name="${prefix}_uleg_root">
@@ -17,4 +23,10 @@
         </geometry>
       </visual>
+      <collision>
+        <origin rpy="0 0 0" xyz="0 0 0"/>
+        <geometry>
+          <mesh filename="package://premaidai_description/meshes/${prefix}_uleg_root.dae"/>
+        </geometry>
+      </collision>
     </link>
     <link name="${prefix}_uleg">
@@ -25,4 +37,10 @@
         </geometry>
       </visual>
+      <collision>
+        <origin rpy="0 0 0" xyz="0 0 0"/>
+        <geometry>
+          <mesh filename="package://premaidai_description/meshes/${prefix}_uleg.dae"/>
+        </geometry>
+      </collision>
     </link>
     <link name="${prefix}_lleg">
@@ -33,4 +51,10 @@
         </geometry>
       </visual>
+      <collision>
+        <origin rpy="0 0 0" xyz="0 0 0"/>
+        <geometry>
+          <mesh filename="package://premaidai_description/meshes/${prefix}_lleg.dae"/>
+        </geometry>
+      </collision>
     </link>
     <link name="${prefix}_dummy">
@@ -49,4 +73,10 @@
         </geometry>
       </visual>
+      <collision>
+        <origin rpy="0 0 0" xyz="0 0 0"/>
+        <geometry>
+          <mesh filename="package://premaidai_description/meshes/${prefix}_foot.dae"/>
+        </geometry>
+      </collision>
     </link>
     <joint name="${prefix}_hpz_joint" type="revolute">

Commit message: Add joint limit to arm

File: urdf/arm.urdf.xacro (robot description, xacro)
@@ -81,5 +81,5 @@
       <xacro:insert_block name="origin" />
       <axis xyz="0 1 0"/>
-      <limit lower="${-pi/2.0}" upper="${pi/2.0}" effort="0" velocity="0"/>
+      <limit lower="${-108.0/180.0 * pi}" upper="${128.25/180.0 * pi}" effort="0" velocity="0"/>
       <parent link="${parent}"/>
       <child link="${prefix}_uarm_joint"/>
@@ -88,5 +88,10 @@
       <origin xyz="0 ${sign*0.0189} 0" rpy="0 0 0"/>
       <axis xyz="1 0 0"/>
-      <limit lower="${-pi / 2.0}" upper="${pi / 2.0}" effort="0" velocity="0"/>
+      <xacro:if value="${side=='right'}">
+        <limit lower="${-3.0375/180.0 * pi}" upper="${91.56375/180.0 * pi}" effort="0" velocity="0"/>
+      </xacro:if>
+      <xacro:if value="${side=='left'}">
+        <limit lower="${-91.56375/180.0 * pi}" upper="${3.0375/180.0 * pi}" effort="0" velocity="0"/>
+      </xacro:if>
       <parent link="${prefix}_uarm_joint"/>
       <child link="${prefix}_uarm"/>
@@ -95,5 +100,5 @@
       <origin xyz="0.0088013 ${sign*0.060007} 0" rpy="0 0 0"/>
       <axis xyz="0 1 0"/>
-      <limit lower="${-pi/2.0}" upper="${pi/2.0}" effort="0" velocity="0"/>
+      <limit lower="${-128.68875/180.0 * pi}" upper="${134.325/180.0 * pi}" effort="0" velocity="0"/>
       <parent link="${prefix}_uarm"/>
       <child link="${prefix}_larm_joint"/>
@@ -102,5 +107,10 @@
       <origin xyz="0 ${sign*0.024054} 0" rpy="0 0 0"/>
       <axis xyz="1 0 0"/>
-      <limit lower="${-pi/2.0}" upper="${pi/2.0}" effort="0" velocity="0"/>
+      <xacro:if value="${side=='right'}">
+        <limit lower="${-13.5/180.0 * pi}" upper="${118.96875/180.0 * pi}" effort="0" velocity="0"/>
+      </xacro:if>
+      <xacro:if value="${side=='left'}">
+        <limit lower="${-118.96875/180.0 * pi}" upper="${13.5/180.0 * pi}" effort="0" velocity="0"/>
+      </xacro:if>
       <parent link="${prefix}_larm_joint"/>
       <child link="${prefix}_larm"/>
@@ -109,5 +119,5 @@
       <origin xyz="0 ${sign*0.061348} 0" rpy="0 0 0"/>
       <axis xyz="0 1 0"/>
-      <limit lower="${-pi/2.0}" upper="${pi/2.0}" effort="0" velocity="0"/>
+      <limit lower="${-135.0/180.0 * pi}" upper="${118.125/180.0 * pi}" effort="0" velocity="0"/>
       <parent link="${prefix}_larm"/>
       <child link="${prefix}_hand"/>

Commit message: Fix model scale

File: urdf/arm.urdf.xacro (robot description, xacro)
@@ -12,5 +12,5 @@
         <origin rpy="0 0 0" xyz="0 0 0"/>
         <geometry>
-          <mesh filename="package://premaidai_description/meshes/${prefix}_uarm_joint.dae" scale="0.01 0.01 0.01"/>
+          <mesh filename="package://premaidai_description/meshes/${prefix}_uarm_joint.dae"/>
         </geometry>
       </visual>
@@ -18,5 +18,5 @@
         <origin rpy="0 0 0" xyz="0 0 0"/>
         <geometry>
-          <mesh filename="package://premaidai_description/meshes/${prefix}_uarm_joint.dae" scale="0.01 0.01 0.01"/>
+          <mesh filename="package://premaidai_description/meshes/${prefix}_uarm_joint.dae"/>
         </geometry>
       </collision>
@@ -26,5 +26,5 @@
         <origin rpy="0 0 0" xyz="0 0 0"/>
         <geometry>
-          <mesh filename="package://premaidai_description/meshes/${prefix}_uarm.dae" scale="0.01 0.01 0.01"/>
+          <mesh filename="package://premaidai_description/meshes/${prefix}_uarm.dae"/>
         </geometry>
       </visual>
@@ -32,5 +32,5 @@
         <origin rpy="0 0 0" xyz="0 0 0"/>
         <geometry>
-          <mesh filename="package://premaidai_description/meshes/${prefix}_uarm.dae" scale="0.01 0.01 0.01"/>
+          <mesh filename="package://premaidai_description/meshes/${prefix}_uarm.dae"/>
         </geometry>
       </collision>
@@ -40,5 +40,5 @@
         <origin rpy="0 0 0" xyz="0 0 0"/>
         <geometry>
-          <mesh filename="package://premaidai_description/meshes/${prefix}_larm_joint.dae" scale="0.01 0.01 0.01"/>
+          <mesh filename="package://premaidai_description/meshes/${prefix}_larm_joint.dae"/>
         </geometry>
       </visual>
@@ -46,5 +46,5 @@
         <origin rpy="0 0 0" xyz="0 0 0"/>
         <geometry>
-          <mesh filename="package://premaidai_description/meshes/${prefix}_larm_joint.dae" scale="0.01 0.01 0.01"/>
+          <mesh filename="package://premaidai_description/meshes/${prefix}_larm_joint.dae"/>
         </geometry>
       </collision>
@@ -54,5 +54,5 @@
         <origin rpy="0 0 0" xyz="0 0 0"/>
         <geometry>
-          <mesh filename="package://premaidai_description/meshes/${prefix}_larm.dae" scale="0.01 0.01 0.01"/>
+          <mesh filename="package://premaidai_description/meshes/${prefix}_larm.dae"/>
         </geometry>
       </visual>
@@ -60,5 +60,5 @@
         <origin rpy="0 0 0" xyz="0 0 0"/>
         <geometry>
-          <mesh filename="package://premaidai_description/meshes/${prefix}_larm.dae" scale="0.01 0.01 0.01"/>
+          <mesh filename="package://premaidai_description/meshes/${prefix}_larm.dae"/>
         </geometry>
       </collision>
@@ -68,5 +68,5 @@
         <origin rpy="0 0 0" xyz="0 0 0"/>
         <geometry>
-          <mesh filename="package://premaidai_description/meshes/${prefix}_hand.dae" scale="0.01 0.01 0.01"/>
+          <mesh filename="package://premaidai_description/meshes/${prefix}_hand.dae"/>
         </geometry>
       </visual>
@@ -74,5 +74,5 @@
         <origin rpy="0 0 0" xyz="0 0 0"/>
         <geometry>
-          <mesh filename="package://premaidai_description/meshes/${prefix}_hand.dae" scale="0.01 0.01 0.01"/>
+          <mesh filename="package://premaidai_description/meshes/${prefix}_hand.dae"/>
         </geometry>
       </collision>

File: urdf/body.urdf.xacro (robot description, xacro)
@@ -5,10 +5,10 @@
       <visual>
         <geometry>
-          <mesh filename="package://premaidai_description/meshes/body.dae" scale="0.01 0.01 0.01"/>
+          <mesh filename="package://premaidai_description/meshes/body.dae"/>
         </geometry>
       </visual>
       <collision>
         <geometry>
-          <mesh filename="package://premaidai_description/meshes/body.dae" scale="0.01 0.01 0.01"/>
+          <mesh filename="package://premaidai_description/meshes/body.dae"/>
         </geometry>
       </collision>
@@ -17,10 +17,10 @@
       <visual>
         <geometry>
-          <mesh filename="package://premaidai_description/meshes/neck_pitch.dae" scale="0.01 0.01 0.01"/>
+          <mesh filename="package://premaidai_description/meshes/neck_pitch.dae"/>
         </geometry>
       </visual>
       <collision>
         <geometry>
-          <mesh filename="package://premaidai_description/meshes/neck_pitch.dae" scale="0.01 0.01 0.01"/>
+          <mesh filename="package://premaidai_description/meshes/neck_pitch.dae"/>
         </geometry>
       </collision>
@@ -29,10 +29,10 @@
       <visual>
         <geometry>
-          <mesh filename="package://premaidai_description/meshes/neck_yaw.dae" scale="0.01 0.01 0.01"/>
+          <mesh filename="package://premaidai_description/meshes/neck_yaw.dae"/>
         </geometry>
       </visual>
       <collision>
         <geometry>
-          <mesh filename="package://premaidai_description/meshes/neck_yaw.dae" scale="0.01 0.01 0.01"/>
+          <mesh filename="package://premaidai_description/meshes/neck_yaw.dae"/>
         </geometry>
       </collision>
@@ -41,10 +41,10 @@
       <visual>
         <geometry>
-          <mesh filename="package://premaidai_description/meshes/head.dae" scale="0.01 0.01 0.01"/>
+          <mesh filename="package://premaidai_description/meshes/head.dae"/>
         </geometry>
       </visual>
       <collision>
         <geometry>
-          <mesh filename="package://premaidai_description/meshes/head.dae" scale="0.01 0.01 0.01"/>
+          <mesh filename="package://premaidai_description/meshes/head.dae"/>
         </geometry>
       </collision>

File: urdf/leg.urdf.xacro (robot description, xacro)
@@ -12,5 +12,5 @@
         <origin rpy="0 0 0" xyz="0 0 0"/>
         <geometry>
-          <mesh filename="package://premaidai_description/meshes/${prefix}_hip_joint.dae" scale="0.01 0.01 0.01"/>
+          <mesh filename="package://premaidai_description/meshes/${prefix}_hip_joint.dae"/>
         </geometry>
       </visual>
@@ -18,5 +18,5 @@
         <origin rpy="0 0 0" xyz="0 0 0"/>
         <geometry>
-          <mesh filename="package://premaidai_description/meshes/${prefix}_hip_joint.dae" scale="0.01 0.01 0.01"/>
+          <mesh filename="package://premaidai_description/meshes/${prefix}_hip_joint.dae"/>
         </geometry>
       </collision>
@@ -26,5 +26,5 @@
         <origin rpy="0 0 0" xyz="0 0 0"/>
         <geometry>
-          <mesh filename="package://premaidai_description/meshes/${prefix}_uleg_root.dae" scale="0.01 0.01 0.01"/>
+          <mesh filename="package://premaidai_description/meshes/${prefix}_uleg_root.dae"/>
         </geometry>
       </visual>
@@ -32,5 +32,5 @@
         <origin rpy="0 0 0" xyz="0 0 0"/>
         <geometry>
-          <mesh filename="package://premaidai_description/meshes/${prefix}_uleg_root.dae" scale="0.01 0.01 0.01"/>
+          <mesh filename="package://premaidai_description/meshes/${prefix}_uleg_root.dae"/>
         </geometry>
       </collision>
@@ -40,5 +40,5 @@
         <origin rpy="0 0 0" xyz="0 0 0"/>
         <geometry>
-          <mesh filename="package://premaidai_description/meshes/${prefix}_uleg.dae" scale="0.01 0.01 0.01"/>
+          <mesh filename="package://premaidai_description/meshes/${prefix}_uleg.dae"/>
         </geometry>
       </visual>
@@ -46,5 +46,5 @@
         <origin rpy="0 0 0" xyz="0 0 0"/>
         <geometry>
-          <mesh filename="package://premaidai_description/meshes/${prefix}_uleg.dae" scale="0.01 0.01 0.01"/>
+          <mesh filename="package://premaidai_description/meshes/${prefix}_uleg.dae"/>
         </geometry>
       </collision>
@@ -54,5 +54,5 @@
         <origin rpy="0 0 0" xyz="0 0 0"/>
         <geometry>
-          <mesh filename="package://premaidai_description/meshes/${prefix}_lleg.dae" scale="0.01 0.01 0.01"/>
+          <mesh filename="package://premaidai_description/meshes/${prefix}_lleg.dae"/>
         </geometry>
       </visual>
@@ -60,5 +60,5 @@
         <origin rpy="0 0 0" xyz="0 0 0"/>
         <geometry>
-          <mesh filename="package://premaidai_description/meshes/${prefix}_lleg.dae" scale="0.01 0.01 0.01"/>
+          <mesh filename="package://premaidai_description/meshes/${prefix}_lleg.dae"/>
         </geometry>
       </collision>
@@ -68,5 +68,5 @@
         <origin rpy="0 0 0" xyz="0 0 0"/>
         <geometry>
-          <mesh filename="package://premaidai_description/meshes/${prefix}_ankle.dae" scale="0.01 0.01 0.01"/>
+          <mesh filename="package://premaidai_description/meshes/${prefix}_ankle.dae"/>
         </geometry>
       </visual>
@@ -74,5 +74,5 @@
         <origin rpy="0 0 0" xyz="0 0 0"/>
         <geometry>
-          <mesh filename="package://premaidai_description/meshes/${prefix}_ankle.dae" scale="0.01 0.01 0.01"/>
+          <mesh filename="package://premaidai_description/meshes/${prefix}_ankle.dae"/>
         </geometry>
       </collision>
@@ -82,5 +82,5 @@
         <origin rpy="0 0 0" xyz="0 0 0"/>
         <geometry>
-          <mesh filename="package://premaidai_description/meshes/${prefix}_foot.dae" scale="0.01 0.01 0.01"/>
+          <mesh filename="package://premaidai_description/meshes/${prefix}_foot.dae"/>
         </geometry>
       </visual>
@@ -88,5 +88,5 @@
         <origin rpy="0 0 0" xyz="0 0 0"/>
         <geometry>
-          <mesh filename="package://premaidai_description/meshes/${prefix}_foot.dae" scale="0.01 0.01 0.01"/>
+          <mesh filename="package://premaidai_description/meshes/${prefix}_foot.dae"/>
         </geometry>
       </collision>
