Commit message: edit velocity and add damping settings.
edit velocity and add damping settings.

File: urdf/arm.urdf.xacro (robot description, xacro)
@@ -114,7 +114,8 @@
       <xacro:insert_block name="origin" />
       <axis xyz="0 1 0"/>
-      <limit lower="${-108.0/180.0 * pi}" upper="${128.25/180.0 * pi}" effort="10" velocity="1.0"/>
+      <limit lower="${-108.0/180.0 * pi}" upper="${128.25/180.0 * pi}" effort="10" velocity="10.0"/>
       <parent link="${parent}"/>
       <child link="${prefix}_uarm_joint"/>
+      <dynamics damping="0.95"/>
     </joint>
     <joint name="${prefix}_shx_joint" type="revolute">
@@ -122,18 +123,20 @@
       <axis xyz="1 0 0"/>
       <xacro:if value="${side=='right'}">
-        <limit lower="${-3.0375/180.0 * pi}" upper="${91.56375/180.0 * pi}" effort="10" velocity="1.0"/>
+        <limit lower="${-3.0375/180.0 * pi}" upper="${91.56375/180.0 * pi}" effort="10" velocity="10.0"/>
       </xacro:if>
       <xacro:if value="${side=='left'}">
-        <limit lower="${-91.56375/180.0 * pi}" upper="${3.0375/180.0 * pi}" effort="10" velocity="1.0"/>
+        <limit lower="${-91.56375/180.0 * pi}" upper="${3.0375/180.0 * pi}" effort="10" velocity="10.0"/>
       </xacro:if>
       <parent link="${prefix}_uarm_joint"/>
       <child link="${prefix}_uarm"/>
+      <dynamics damping="0.95"/>
     </joint>
     <joint name="${prefix}_ely_joint" type="revolute">
       <origin xyz="0.0088013 ${sign*0.060007} 0" rpy="0 0 0"/>
       <axis xyz="0 1 0"/>
-      <limit lower="${-128.68875/180.0 * pi}" upper="${134.325/180.0 * pi}" effort="10" velocity="1.0"/>
+      <limit lower="${-128.68875/180.0 * pi}" upper="${134.325/180.0 * pi}" effort="10" velocity="10.0"/>
       <parent link="${prefix}_uarm"/>
       <child link="${prefix}_larm_joint"/>
+      <dynamics damping="0.95"/>
     </joint>
     <joint name="${prefix}_elx_joint" type="revolute">
@@ -141,18 +144,20 @@
       <axis xyz="1 0 0"/>
       <xacro:if value="${side=='right'}">
-        <limit lower="${-13.5/180.0 * pi}" upper="${118.96875/180.0 * pi}" effort="10" velocity="1.0"/>
+        <limit lower="${-13.5/180.0 * pi}" upper="${118.96875/180.0 * pi}" effort="10" velocity="10.0"/>
       </xacro:if>
       <xacro:if value="${side=='left'}">
-        <limit lower="${-118.96875/180.0 * pi}" upper="${13.5/180.0 * pi}" effort="10" velocity="1.0"/>
+        <limit lower="${-118.96875/180.0 * pi}" upper="${13.5/180.0 * pi}" effort="10" velocity="10.0"/>
       </xacro:if>
       <parent link="${prefix}_larm_joint"/>
       <child link="${prefix}_larm"/>
+      <dynamics damping="0.95"/>
     </joint>
     <joint name="${prefix}_wry_joint" type="revolute">
       <origin xyz="0 ${sign*0.061348} 0" rpy="0 0 0"/>
       <axis xyz="0 1 0"/>
-      <limit lower="${-135.0/180.0 * pi}" upper="${118.125/180.0 * pi}" effort="10" velocity="1.0"/>
+      <limit lower="${-135.0/180.0 * pi}" upper="${118.125/180.0 * pi}" effort="10" velocity="10.0"/>
       <parent link="${prefix}_larm"/>
       <child link="${prefix}_hand"/>
+      <dynamics damping="0.95"/>
     </joint>
     <joint name="${prefix}_hand_ee_fixed_joint" type="fixed">
@@ -160,4 +165,5 @@
       <child link = "${prefix}_hand_ee" />
       <origin xyz="0.0 0.0 0.0" rpy="0.0 0.0 0.0" />
+      <dynamics damping="0.95"/>
     </joint>
   </xacro:macro>

File: urdf/body.urdf.xacro (robot description, xacro)
@@ -74,25 +74,29 @@
       <parent link="${parent}"/>
       <child link="body"/>
+      <dynamics damping="0.95"/>
     </joint>
     <joint name="head_ny_joint" type="revolute">
       <origin xyz="0.0038738 0 0.132809" rpy="0 0 0"/>
       <axis xyz="0 1 0"/>
-      <limit lower="${-10.125/180.0 * pi}" upper="${23.625/180.0 * pi}" effort="10" velocity="1.0"/>
+      <limit lower="${-10.125/180.0 * pi}" upper="${23.625/180.0 * pi}" effort="10" velocity="10.0"/>
       <parent link="body"/>
       <child link="neck_pitch"/>
+      <dynamics damping="0.95"/>
     </joint>
     <joint name="head_nz_joint" type="revolute">
       <origin xyz="-0.0103485 0 0.011103" rpy="0 0 0"/>
       <axis xyz="0 0 1"/>
-      <limit lower="${-47.25/180.0 * pi}" upper="${47.25/180.0 * pi}" effort="10" velocity="1.0"/>
+      <limit lower="${-47.25/180.0 * pi}" upper="${47.25/180.0 * pi}" effort="10" velocity="10.0"/>
       <parent link="neck_pitch"/>
       <child link="head_yaw"/>
+      <dynamics damping="0.95"/>
     </joint>
     <joint name="head_nx_joint" type="revolute">
       <origin xyz="0 0 0.0129" rpy="0 0 0"/>
       <axis xyz="1 0 0"/>
-      <limit lower="${-21.9375/180.0 * pi}" upper="${28.6875/180.0 * pi}" effort="10" velocity="1.0"/>
+      <limit lower="${-21.9375/180.0 * pi}" upper="${28.6875/180.0 * pi}" effort="10" velocity="10.0"/>
       <parent link="head_yaw"/>
       <child link="head"/>
+      <dynamics damping="0.95"/>
     </joint>
   </xacro:macro>

File: urdf/leg.urdf.xacro (robot description, xacro)
@@ -125,7 +125,8 @@
       <xacro:insert_block name="origin" />
       <axis xyz="0 0 1"/>
-      <limit lower="${-81.0/180.0 * pi}" upper="${102.43/180.0 * pi}" effort="10" velocity="1.0"/>
+      <limit lower="${-81.0/180.0 * pi}" upper="${102.43/180.0 * pi}" effort="10" velocity="10.0"/>
       <parent link="${parent}"/>
       <child link="${prefix}_hip_joint"/>
+      <dynamics damping="0.95"/>
     </joint>
     <joint name="${prefix}_hpx_joint" type="revolute">
@@ -133,32 +134,36 @@
       <axis xyz="1 0 0"/>
       <xacro:if value="${side=='right'}">
-        <limit lower="${-25.35/180.0 * pi}" upper="${22.713/180.0 * pi}" effort="10" velocity="1.0"/>
+        <limit lower="${-25.35/180.0 * pi}" upper="${22.713/180.0 * pi}" effort="10" velocity="10.0"/>
       </xacro:if>
       <xacro:if value="${side=='left'}">
-        <limit lower="${-22.713/180.0 * pi}" upper="${25.35/180.0 * pi}" effort="10" velocity="1.0"/>
+        <limit lower="${-22.713/180.0 * pi}" upper="${25.35/180.0 * pi}" effort="10" velocity="10.0"/>
       </xacro:if>
       <parent link="${prefix}_hip_joint"/>
       <child link="${prefix}_uleg_root"/>
+      <dynamics damping="0.95"/>
     </joint>
     <joint name="${prefix}_hpy_joint" type="revolute">
       <origin xyz="0 ${sign*0.0128525} -0.034358" rpy="0 0 0"/>
       <axis xyz="0 1 0"/>
-      <limit lower="${-91.60/180.0 * pi}" upper="${90.213/180.0 * pi}" effort="10" velocity="1.0"/>
+      <limit lower="${-91.60/180.0 * pi}" upper="${90.213/180.0 * pi}" effort="10" velocity="10.0"/>
       <parent link="${prefix}_uleg_root"/>
       <child link="${prefix}_uleg"/>
+      <dynamics damping="0.95"/>
     </joint>
     <joint name="${prefix}_kny_joint" type="revolute">
       <origin xyz="0 0 -0.0652" rpy="0 0 0"/>
       <axis xyz="0 1 0"/>
-      <limit lower="${-2.0925/180.0 * pi}" upper="${119.64/180.0 * pi}" effort="10" velocity="1.0"/>
+      <limit lower="${-2.0925/180.0 * pi}" upper="${119.64/180.0 * pi}" effort="10" velocity="10.0"/>
       <parent link="${prefix}_uleg"/>
       <child link="${prefix}_lleg"/>
+      <dynamics damping="0.95"/>
     </joint>
     <joint name="${prefix}_aky_joint" type="revolute">
       <origin xyz="0 0 -0.065" rpy="0 0 0"/>
       <axis xyz="0 1 0"/>
-      <limit lower="${-61.3575/180.0 * pi}" upper="${24.3/180.0 * pi}" effort="10" velocity="1.0"/>
+      <limit lower="${-61.3575/180.0 * pi}" upper="${24.3/180.0 * pi}" effort="10" velocity="10.0"/>
       <parent link="${prefix}_lleg"/>
       <child link="${prefix}_ankle"/>
+      <dynamics damping="0.95"/>
     </joint>
     <joint name="${prefix}_akx_joint" type="revolute">
@@ -166,11 +171,12 @@
       <axis xyz="1 0 0"/>
       <xacro:if value="${side=='right'}">
-        <limit lower="${-38.23875/180.0 * pi}" upper="${37.29375/180.0 * pi}" effort="10" velocity="1.0"/>
+        <limit lower="${-38.23875/180.0 * pi}" upper="${37.29375/180.0 * pi}" effort="10" velocity="10.0"/>
       </xacro:if>
       <xacro:if value="${side=='left'}">
-        <limit lower="${-37.29375/180.0 * pi}" upper="${38.23875/180.0 * pi}" effort="10" velocity="1.0"/>
+        <limit lower="${-37.29375/180.0 * pi}" upper="${38.23875/180.0 * pi}" effort="10" velocity="10.0"/>
       </xacro:if>
       <parent link="${prefix}_ankle"/>
       <child link="${prefix}_foot"/>
+      <dynamics damping="0.95"/>
     </joint>
   </xacro:macro>

Commit message: Update joint velocity limit values

File: urdf/arm.urdf.xacro (robot description, xacro)
@@ -114,5 +114,5 @@
       <xacro:insert_block name="origin" />
       <axis xyz="0 1 0"/>
-      <limit lower="${-108.0/180.0 * pi}" upper="${128.25/180.0 * pi}" effort="10" velocity="1.0"/>
+      <limit lower="${-108.0/180.0 * pi}" upper="${128.25/180.0 * pi}" effort="10" velocity="7.480"/>
       <parent link="${parent}"/>
       <child link="${prefix}_uarm_joint"/>
@@ -122,8 +122,8 @@
       <axis xyz="1 0 0"/>
       <xacro:if value="${side=='right'}">
-        <limit lower="${-3.0375/180.0 * pi}" upper="${91.56375/180.0 * pi}" effort="10" velocity="1.0"/>
+        <limit lower="${-3.0375/180.0 * pi}" upper="${91.56375/180.0 * pi}" effort="10" velocity="5.817"/>
       </xacro:if>
       <xacro:if value="${side=='left'}">
-        <limit lower="${-91.56375/180.0 * pi}" upper="${3.0375/180.0 * pi}" effort="10" velocity="1.0"/>
+        <limit lower="${-91.56375/180.0 * pi}" upper="${3.0375/180.0 * pi}" effort="10" velocity="5.817"/>
       </xacro:if>
       <parent link="${prefix}_uarm_joint"/>
@@ -133,5 +133,5 @@
       <origin xyz="0.0088013 ${sign*0.060007} 0" rpy="0 0 0"/>
       <axis xyz="0 1 0"/>
-      <limit lower="${-128.68875/180.0 * pi}" upper="${134.325/180.0 * pi}" effort="10" velocity="1.0"/>
+      <limit lower="${-128.68875/180.0 * pi}" upper="${134.325/180.0 * pi}" effort="10" velocity="5.817"/>
       <parent link="${prefix}_uarm"/>
       <child link="${prefix}_larm_joint"/>
@@ -141,8 +141,8 @@
       <axis xyz="1 0 0"/>
       <xacro:if value="${side=='right'}">
-        <limit lower="${-13.5/180.0 * pi}" upper="${118.96875/180.0 * pi}" effort="10" velocity="1.0"/>
+        <limit lower="${-13.5/180.0 * pi}" upper="${118.96875/180.0 * pi}" effort="10" velocity="5.817"/>
       </xacro:if>
       <xacro:if value="${side=='left'}">
-        <limit lower="${-118.96875/180.0 * pi}" upper="${13.5/180.0 * pi}" effort="10" velocity="1.0"/>
+        <limit lower="${-118.96875/180.0 * pi}" upper="${13.5/180.0 * pi}" effort="10" velocity="5.817"/>
       </xacro:if>
       <parent link="${prefix}_larm_joint"/>
@@ -152,5 +152,5 @@
       <origin xyz="0 ${sign*0.061348} 0" rpy="0 0 0"/>
       <axis xyz="0 1 0"/>
-      <limit lower="${-135.0/180.0 * pi}" upper="${118.125/180.0 * pi}" effort="10" velocity="1.0"/>
+      <limit lower="${-135.0/180.0 * pi}" upper="${118.125/180.0 * pi}" effort="10" velocity="5.817"/>
       <parent link="${prefix}_larm"/>
       <child link="${prefix}_hand"/>

File: urdf/body.urdf.xacro (robot description, xacro)
@@ -78,5 +78,5 @@
       <origin xyz="0.0038738 0 0.132809" rpy="0 0 0"/>
       <axis xyz="0 1 0"/>
-      <limit lower="${-10.125/180.0 * pi}" upper="${23.625/180.0 * pi}" effort="10" velocity="1.0"/>
+      <limit lower="${-10.125/180.0 * pi}" upper="${23.625/180.0 * pi}" effort="10" velocity="5.817"/>
       <parent link="body"/>
       <child link="neck_pitch"/>
@@ -85,5 +85,5 @@
       <origin xyz="-0.0103485 0 0.011103" rpy="0 0 0"/>
       <axis xyz="0 0 1"/>
-      <limit lower="${-47.25/180.0 * pi}" upper="${47.25/180.0 * pi}" effort="10" velocity="1.0"/>
+      <limit lower="${-47.25/180.0 * pi}" upper="${47.25/180.0 * pi}" effort="10" velocity="5.817"/>
       <parent link="neck_pitch"/>
       <child link="head_yaw"/>
@@ -92,5 +92,5 @@
       <origin xyz="0 0 0.0129" rpy="0 0 0"/>
       <axis xyz="1 0 0"/>
-      <limit lower="${-21.9375/180.0 * pi}" upper="${28.6875/180.0 * pi}" effort="10" velocity="1.0"/>
+      <limit lower="${-21.9375/180.0 * pi}" upper="${28.6875/180.0 * pi}" effort="10" velocity="5.817"/>
       <parent link="head_yaw"/>
       <child link="head"/>

File: urdf/leg.urdf.xacro (robot description, xacro)
@@ -125,5 +125,5 @@
       <xacro:insert_block name="origin" />
       <axis xyz="0 0 1"/>
-      <limit lower="${-81.0/180.0 * pi}" upper="${102.43/180.0 * pi}" effort="10" velocity="1.0"/>
+      <limit lower="${-81.0/180.0 * pi}" upper="${102.43/180.0 * pi}" effort="10" velocity="7.480"/>
       <parent link="${parent}"/>
       <child link="${prefix}_hip_joint"/>
@@ -133,8 +133,8 @@
       <axis xyz="1 0 0"/>
       <xacro:if value="${side=='right'}">
-        <limit lower="${-25.35/180.0 * pi}" upper="${22.713/180.0 * pi}" effort="10" velocity="1.0"/>
+        <limit lower="${-25.35/180.0 * pi}" upper="${22.713/180.0 * pi}" effort="10" velocity="7.480"/>
       </xacro:if>
       <xacro:if value="${side=='left'}">
-        <limit lower="${-22.713/180.0 * pi}" upper="${25.35/180.0 * pi}" effort="10" velocity="1.0"/>
+        <limit lower="${-22.713/180.0 * pi}" upper="${25.35/180.0 * pi}" effort="10" velocity="7.480"/>
       </xacro:if>
       <parent link="${prefix}_hip_joint"/>
@@ -144,5 +144,5 @@
       <origin xyz="0 ${sign*0.0128525} -0.034358" rpy="0 0 0"/>
       <axis xyz="0 1 0"/>
-      <limit lower="${-91.60/180.0 * pi}" upper="${90.213/180.0 * pi}" effort="10" velocity="1.0"/>
+      <limit lower="${-91.60/180.0 * pi}" upper="${90.213/180.0 * pi}" effort="10" velocity="7.480"/>
       <parent link="${prefix}_uleg_root"/>
       <child link="${prefix}_uleg"/>
@@ -151,5 +151,5 @@
       <origin xyz="0 0 -0.0652" rpy="0 0 0"/>
       <axis xyz="0 1 0"/>
-      <limit lower="${-2.0925/180.0 * pi}" upper="${119.64/180.0 * pi}" effort="10" velocity="1.0"/>
+      <limit lower="${-2.0925/180.0 * pi}" upper="${119.64/180.0 * pi}" effort="10" velocity="7.480"/>
       <parent link="${prefix}_uleg"/>
       <child link="${prefix}_lleg"/>
@@ -158,5 +158,5 @@
       <origin xyz="0 0 -0.065" rpy="0 0 0"/>
       <axis xyz="0 1 0"/>
-      <limit lower="${-61.3575/180.0 * pi}" upper="${24.3/180.0 * pi}" effort="10" velocity="1.0"/>
+      <limit lower="${-61.3575/180.0 * pi}" upper="${24.3/180.0 * pi}" effort="10" velocity="7.480"/>
       <parent link="${prefix}_lleg"/>
       <child link="${prefix}_ankle"/>
@@ -166,8 +166,8 @@
       <axis xyz="1 0 0"/>
       <xacro:if value="${side=='right'}">
-        <limit lower="${-38.23875/180.0 * pi}" upper="${37.29375/180.0 * pi}" effort="10" velocity="1.0"/>
+        <limit lower="${-38.23875/180.0 * pi}" upper="${37.29375/180.0 * pi}" effort="10" velocity="7.480"/>
       </xacro:if>
       <xacro:if value="${side=='left'}">
-        <limit lower="${-37.29375/180.0 * pi}" upper="${38.23875/180.0 * pi}" effort="10" velocity="1.0"/>
+        <limit lower="${-37.29375/180.0 * pi}" upper="${38.23875/180.0 * pi}" effort="10" velocity="7.480"/>
       </xacro:if>
       <parent link="${prefix}_ankle"/>

Commit message: Add joint damping values

File: urdf/arm.urdf.xacro (robot description, xacro)
@@ -115,4 +115,5 @@
       <axis xyz="0 1 0"/>
       <limit lower="${-108.0/180.0 * pi}" upper="${128.25/180.0 * pi}" effort="10" velocity="7.480"/>
+      <dynamics damping="0.4" friction="0.0"/>
       <parent link="${parent}"/>
       <child link="${prefix}_uarm_joint"/>
@@ -127,4 +128,5 @@
         <limit lower="${-91.56375/180.0 * pi}" upper="${3.0375/180.0 * pi}" effort="10" velocity="5.817"/>
       </xacro:if>
+      <dynamics damping="0.4" friction="0.0"/>
       <parent link="${prefix}_uarm_joint"/>
       <child link="${prefix}_uarm"/>
@@ -134,4 +136,5 @@
       <axis xyz="0 1 0"/>
       <limit lower="${-128.68875/180.0 * pi}" upper="${134.325/180.0 * pi}" effort="10" velocity="5.817"/>
+      <dynamics damping="0.4" friction="0.0"/>
       <parent link="${prefix}_uarm"/>
       <child link="${prefix}_larm_joint"/>
@@ -146,4 +149,5 @@
         <limit lower="${-118.96875/180.0 * pi}" upper="${13.5/180.0 * pi}" effort="10" velocity="5.817"/>
       </xacro:if>
+      <dynamics damping="0.4" friction="0.0"/>
       <parent link="${prefix}_larm_joint"/>
       <child link="${prefix}_larm"/>
@@ -153,4 +157,5 @@
       <axis xyz="0 1 0"/>
       <limit lower="${-135.0/180.0 * pi}" upper="${118.125/180.0 * pi}" effort="10" velocity="5.817"/>
+      <dynamics damping="0.4" friction="0.0"/>
       <parent link="${prefix}_larm"/>
       <child link="${prefix}_hand"/>

File: urdf/body.urdf.xacro (robot description, xacro)
@@ -79,4 +79,5 @@
       <axis xyz="0 1 0"/>
       <limit lower="${-10.125/180.0 * pi}" upper="${23.625/180.0 * pi}" effort="10" velocity="5.817"/>
+      <dynamics damping="0.4" friction="0.0"/>
       <parent link="body"/>
       <child link="neck_pitch"/>
@@ -86,4 +87,5 @@
       <axis xyz="0 0 1"/>
       <limit lower="${-47.25/180.0 * pi}" upper="${47.25/180.0 * pi}" effort="10" velocity="5.817"/>
+      <dynamics damping="0.4" friction="0.0"/>
       <parent link="neck_pitch"/>
       <child link="head_yaw"/>
@@ -93,4 +95,5 @@
       <axis xyz="1 0 0"/>
       <limit lower="${-21.9375/180.0 * pi}" upper="${28.6875/180.0 * pi}" effort="10" velocity="5.817"/>
+      <dynamics damping="0.4" friction="0.0"/>
       <parent link="head_yaw"/>
       <child link="head"/>

File: urdf/leg.urdf.xacro (robot description, xacro)
@@ -126,4 +126,5 @@
       <axis xyz="0 0 1"/>
       <limit lower="${-81.0/180.0 * pi}" upper="${102.43/180.0 * pi}" effort="10" velocity="7.480"/>
+      <dynamics damping="0.4" friction="0.0"/>
       <parent link="${parent}"/>
       <child link="${prefix}_hip_joint"/>
@@ -138,4 +139,5 @@
         <limit lower="${-22.713/180.0 * pi}" upper="${25.35/180.0 * pi}" effort="10" velocity="7.480"/>
       </xacro:if>
+      <dynamics damping="0.4" friction="0.0"/>
       <parent link="${prefix}_hip_joint"/>
       <child link="${prefix}_uleg_root"/>
@@ -145,4 +147,5 @@
       <axis xyz="0 1 0"/>
       <limit lower="${-91.60/180.0 * pi}" upper="${90.213/180.0 * pi}" effort="10" velocity="7.480"/>
+      <dynamics damping="0.4" friction="0.0"/>
       <parent link="${prefix}_uleg_root"/>
       <child link="${prefix}_uleg"/>
@@ -152,4 +155,5 @@
       <axis xyz="0 1 0"/>
       <limit lower="${-2.0925/180.0 * pi}" upper="${119.64/180.0 * pi}" effort="10" velocity="7.480"/>
+      <dynamics damping="0.4" friction="0.0"/>
       <parent link="${prefix}_uleg"/>
       <child link="${prefix}_lleg"/>
@@ -159,4 +163,5 @@
       <axis xyz="0 1 0"/>
       <limit lower="${-61.3575/180.0 * pi}" upper="${24.3/180.0 * pi}" effort="10" velocity="7.480"/>
+      <dynamics damping="0.4" friction="0.0"/>
       <parent link="${prefix}_lleg"/>
       <child link="${prefix}_ankle"/>
@@ -171,4 +176,5 @@
         <limit lower="${-37.29375/180.0 * pi}" upper="${38.23875/180.0 * pi}" effort="10" velocity="7.480"/>
       </xacro:if>
+      <dynamics damping="0.4" friction="0.0"/>
       <parent link="${prefix}_ankle"/>
       <child link="${prefix}_foot"/>
