Commit message: Fix servo effort value

File: urdf/arm.urdf.xacro (robot description, xacro)
@@ -114,5 +114,5 @@
       <xacro:insert_block name="origin" />
       <axis xyz="0 1 0"/>
-      <limit lower="${-108.0/180.0 * pi}" upper="${128.25/180.0 * pi}" effort="10" velocity="7.480"/>
+      <limit lower="${-108.0/180.0 * pi}" upper="${128.25/180.0 * pi}" effort="1.3712" velocity="7.480"/>
       <dynamics damping="0.4" friction="0.0"/>
       <parent link="${parent}"/>
@@ -123,8 +123,8 @@
       <axis xyz="1 0 0"/>
       <xacro:if value="${side=='right'}">
-        <limit lower="${-3.0375/180.0 * pi}" upper="${91.56375/180.0 * pi}" effort="10" velocity="5.817"/>
+        <limit lower="${-3.0375/180.0 * pi}" upper="${91.56375/180.0 * pi}" effort="0.735" velocity="5.817"/>
       </xacro:if>
       <xacro:if value="${side=='left'}">
-        <limit lower="${-91.56375/180.0 * pi}" upper="${3.0375/180.0 * pi}" effort="10" velocity="5.817"/>
+        <limit lower="${-91.56375/180.0 * pi}" upper="${3.0375/180.0 * pi}" effort="0.735" velocity="5.817"/>
       </xacro:if>
       <dynamics damping="0.4" friction="0.0"/>
@@ -135,5 +135,5 @@
       <origin xyz="0.0088013 ${sign*0.060007} 0" rpy="0 0 0"/>
       <axis xyz="0 1 0"/>
-      <limit lower="${-128.68875/180.0 * pi}" upper="${134.325/180.0 * pi}" effort="10" velocity="5.817"/>
+      <limit lower="${-128.68875/180.0 * pi}" upper="${134.325/180.0 * pi}" effort="0.735" velocity="5.817"/>
       <dynamics damping="0.4" friction="0.0"/>
       <parent link="${prefix}_uarm"/>
@@ -144,8 +144,8 @@
       <axis xyz="1 0 0"/>
       <xacro:if value="${side=='right'}">
-        <limit lower="${-13.5/180.0 * pi}" upper="${118.96875/180.0 * pi}" effort="10" velocity="5.817"/>
+        <limit lower="${-13.5/180.0 * pi}" upper="${118.96875/180.0 * pi}" effort="0.735" velocity="5.817"/>
       </xacro:if>
       <xacro:if value="${side=='left'}">
-        <limit lower="${-118.96875/180.0 * pi}" upper="${13.5/180.0 * pi}" effort="10" velocity="5.817"/>
+        <limit lower="${-118.96875/180.0 * pi}" upper="${13.5/180.0 * pi}" effort="0.735" velocity="5.817"/>
       </xacro:if>
       <dynamics damping="0.4" friction="0.0"/>
@@ -156,5 +156,5 @@
       <origin xyz="0 ${sign*0.061348} 0" rpy="0 0 0"/>
       <axis xyz="0 1 0"/>
-      <limit lower="${-135.0/180.0 * pi}" upper="${118.125/180.0 * pi}" effort="10" velocity="5.817"/>
+      <limit lower="${-135.0/180.0 * pi}" upper="${118.125/180.0 * pi}" effort="0.735" velocity="5.817"/>
       <dynamics damping="0.4" friction="0.0"/>
       <parent link="${prefix}_larm"/>

File: urdf/body.urdf.xacro (robot description, xacro)
@@ -78,5 +78,5 @@
       <origin xyz="0.0038738 0 0.132809" rpy="0 0 0"/>
       <axis xyz="0 1 0"/>
-      <limit lower="${-10.125/180.0 * pi}" upper="${23.625/180.0 * pi}" effort="10" velocity="5.817"/>
+      <limit lower="${-10.125/180.0 * pi}" upper="${23.625/180.0 * pi}" effort="0.735" velocity="5.817"/>
       <dynamics damping="0.4" friction="0.0"/>
       <parent link="body"/>
@@ -86,5 +86,5 @@
       <origin xyz="-0.0103485 0 0.011103" rpy="0 0 0"/>
       <axis xyz="0 0 1"/>
-      <limit lower="${-47.25/180.0 * pi}" upper="${47.25/180.0 * pi}" effort="10" velocity="5.817"/>
+      <limit lower="${-47.25/180.0 * pi}" upper="${47.25/180.0 * pi}" effort="0.735" velocity="5.817"/>
       <dynamics damping="0.4" friction="0.0"/>
       <parent link="neck_pitch"/>
@@ -94,5 +94,5 @@
       <origin xyz="0 0 0.0129" rpy="0 0 0"/>
       <axis xyz="1 0 0"/>
-      <limit lower="${-21.9375/180.0 * pi}" upper="${28.6875/180.0 * pi}" effort="10" velocity="5.817"/>
+      <limit lower="${-21.9375/180.0 * pi}" upper="${28.6875/180.0 * pi}" effort="0.735" velocity="5.817"/>
       <dynamics damping="0.4" friction="0.0"/>
       <parent link="head_yaw"/>

File: urdf/leg.urdf.xacro (robot description, xacro)
@@ -125,5 +125,5 @@
       <xacro:insert_block name="origin" />
       <axis xyz="0 0 1"/>
-      <limit lower="${-81.0/180.0 * pi}" upper="${102.43/180.0 * pi}" effort="10" velocity="7.480"/>
+      <limit lower="${-81.0/180.0 * pi}" upper="${102.43/180.0 * pi}" effort="1.3712" velocity="7.480"/>
       <dynamics damping="0.4" friction="0.0"/>
       <parent link="${parent}"/>
@@ -134,8 +134,8 @@
       <axis xyz="1 0 0"/>
       <xacro:if value="${side=='right'}">
-        <limit lower="${-25.35/180.0 * pi}" upper="${22.713/180.0 * pi}" effort="10" velocity="7.480"/>
+        <limit lower="${-25.35/180.0 * pi}" upper="${22.713/180.0 * pi}" effort="1.3712" velocity="7.480"/>
       </xacro:if>
       <xacro:if value="${side=='left'}">
-        <limit lower="${-22.713/180.0 * pi}" upper="${25.35/180.0 * pi}" effort="10" velocity="7.480"/>
+        <limit lower="${-22.713/180.0 * pi}" upper="${25.35/180.0 * pi}" effort="1.3712" velocity="7.480"/>
       </xacro:if>
       <dynamics damping="0.4" friction="0.0"/>
@@ -146,5 +146,5 @@
       <origin xyz="0 ${sign*0.0128525} -0.034358" rpy="0 0 0"/>
       <axis xyz="0 1 0"/>
-      <limit lower="${-91.60/180.0 * pi}" upper="${90.213/180.0 * pi}" effort="10" velocity="7.480"/>
+      <limit lower="${-91.60/180.0 * pi}" upper="${90.213/180.0 * pi}" effort="1.3712" velocity="7.480"/>
       <dynamics damping="0.4" friction="0.0"/>
       <parent link="${prefix}_uleg_root"/>
@@ -154,5 +154,5 @@
       <origin xyz="0 0 -0.0652" rpy="0 0 0"/>
       <axis xyz="0 1 0"/>
-      <limit lower="${-2.0925/180.0 * pi}" upper="${119.64/180.0 * pi}" effort="10" velocity="7.480"/>
+      <limit lower="${-2.0925/180.0 * pi}" upper="${119.64/180.0 * pi}" effort="1.3712" velocity="7.480"/>
       <dynamics damping="0.4" friction="0.0"/>
       <parent link="${prefix}_uleg"/>
@@ -162,5 +162,5 @@
       <origin xyz="0 0 -0.065" rpy="0 0 0"/>
       <axis xyz="0 1 0"/>
-      <limit lower="${-61.3575/180.0 * pi}" upper="${24.3/180.0 * pi}" effort="10" velocity="7.480"/>
+      <limit lower="${-61.3575/180.0 * pi}" upper="${24.3/180.0 * pi}" effort="1.3712" velocity="7.480"/>
       <dynamics damping="0.4" friction="0.0"/>
       <parent link="${prefix}_lleg"/>
@@ -171,8 +171,8 @@
       <axis xyz="1 0 0"/>
       <xacro:if value="${side=='right'}">
-        <limit lower="${-38.23875/180.0 * pi}" upper="${37.29375/180.0 * pi}" effort="10" velocity="7.480"/>
+        <limit lower="${-38.23875/180.0 * pi}" upper="${37.29375/180.0 * pi}" effort="1.3712" velocity="7.480"/>
       </xacro:if>
       <xacro:if value="${side=='left'}">
-        <limit lower="${-37.29375/180.0 * pi}" upper="${38.23875/180.0 * pi}" effort="10" velocity="7.480"/>
+        <limit lower="${-37.29375/180.0 * pi}" upper="${38.23875/180.0 * pi}" effort="1.3712" velocity="7.480"/>
       </xacro:if>
       <dynamics damping="0.4" friction="0.0"/>

Commit message: Update KRS-3224 efforts

File: urdf/arm.urdf.xacro (robot description, xacro)
@@ -123,8 +123,8 @@
       <axis xyz="1 0 0"/>
       <xacro:if value="${side=='right'}">
-        <limit lower="${-3.0375/180.0 * pi}" upper="${91.56375/180.0 * pi}" effort="0.735" velocity="5.817"/>
+        <limit lower="${-3.0375/180.0 * pi}" upper="${91.56375/180.0 * pi}" effort="0.9114" velocity="5.817"/>
       </xacro:if>
       <xacro:if value="${side=='left'}">
-        <limit lower="${-91.56375/180.0 * pi}" upper="${3.0375/180.0 * pi}" effort="0.735" velocity="5.817"/>
+        <limit lower="${-91.56375/180.0 * pi}" upper="${3.0375/180.0 * pi}" effort="0.9114" velocity="5.817"/>
       </xacro:if>
       <dynamics damping="0.4" friction="0.0"/>
@@ -135,5 +135,5 @@
       <origin xyz="0.0088013 ${sign*0.060007} 0" rpy="0 0 0"/>
       <axis xyz="0 1 0"/>
-      <limit lower="${-128.68875/180.0 * pi}" upper="${134.325/180.0 * pi}" effort="0.735" velocity="5.817"/>
+      <limit lower="${-128.68875/180.0 * pi}" upper="${134.325/180.0 * pi}" effort="0.9114" velocity="5.817"/>
       <dynamics damping="0.4" friction="0.0"/>
       <parent link="${prefix}_uarm"/>
@@ -144,8 +144,8 @@
       <axis xyz="1 0 0"/>
       <xacro:if value="${side=='right'}">
-        <limit lower="${-13.5/180.0 * pi}" upper="${118.96875/180.0 * pi}" effort="0.735" velocity="5.817"/>
+        <limit lower="${-13.5/180.0 * pi}" upper="${118.96875/180.0 * pi}" effort="0.9114" velocity="5.817"/>
       </xacro:if>
       <xacro:if value="${side=='left'}">
-        <limit lower="${-118.96875/180.0 * pi}" upper="${13.5/180.0 * pi}" effort="0.735" velocity="5.817"/>
+        <limit lower="${-118.96875/180.0 * pi}" upper="${13.5/180.0 * pi}" effort="0.9114" velocity="5.817"/>
       </xacro:if>
       <dynamics damping="0.4" friction="0.0"/>
@@ -156,5 +156,5 @@
       <origin xyz="0 ${sign*0.061348} 0" rpy="0 0 0"/>
       <axis xyz="0 1 0"/>
-      <limit lower="${-135.0/180.0 * pi}" upper="${118.125/180.0 * pi}" effort="0.735" velocity="5.817"/>
+      <limit lower="${-135.0/180.0 * pi}" upper="${118.125/180.0 * pi}" effort="0.9114" velocity="5.817"/>
       <dynamics damping="0.4" friction="0.0"/>
       <parent link="${prefix}_larm"/>

File: urdf/body.urdf.xacro (robot description, xacro)
@@ -78,5 +78,5 @@
       <origin xyz="0.0038738 0 0.132809" rpy="0 0 0"/>
       <axis xyz="0 1 0"/>
-      <limit lower="${-10.125/180.0 * pi}" upper="${23.625/180.0 * pi}" effort="0.735" velocity="5.817"/>
+      <limit lower="${-10.125/180.0 * pi}" upper="${23.625/180.0 * pi}" effort="0.9114" velocity="5.817"/>
       <dynamics damping="0.4" friction="0.0"/>
       <parent link="body"/>
@@ -86,5 +86,5 @@
       <origin xyz="-0.0103485 0 0.011103" rpy="0 0 0"/>
       <axis xyz="0 0 1"/>
-      <limit lower="${-47.25/180.0 * pi}" upper="${47.25/180.0 * pi}" effort="0.735" velocity="5.817"/>
+      <limit lower="${-47.25/180.0 * pi}" upper="${47.25/180.0 * pi}" effort="0.9114" velocity="5.817"/>
       <dynamics damping="0.4" friction="0.0"/>
       <parent link="neck_pitch"/>
@@ -94,5 +94,5 @@
       <origin xyz="0 0 0.0129" rpy="0 0 0"/>
       <axis xyz="1 0 0"/>
-      <limit lower="${-21.9375/180.0 * pi}" upper="${28.6875/180.0 * pi}" effort="0.735" velocity="5.817"/>
+      <limit lower="${-21.9375/180.0 * pi}" upper="${28.6875/180.0 * pi}" effort="0.9114" velocity="5.817"/>
       <dynamics damping="0.4" friction="0.0"/>
       <parent link="head_yaw"/>
