Commit message: Refactoring urdf files

File: robots/premaidai.urdf.xacro (robot description, xacro)
@@ -3,22 +3,20 @@
   xmlns:xacro="http://ros.org/wiki/xacro">
   <xacro:include filename="$(find premaidai_description)/urdf/common.xacro" />
-  <xacro:include filename="$(find premaidai_description)/urdf/lleg.urdf.xacro" />
-  <xacro:include filename="$(find premaidai_description)/urdf/rleg.urdf.xacro" />
-  <xacro:include filename="$(find premaidai_description)/urdf/larm.urdf.xacro" />
-  <xacro:include filename="$(find premaidai_description)/urdf/rarm.urdf.xacro" />
+  <xacro:include filename="$(find premaidai_description)/urdf/leg.urdf.xacro" />
+  <xacro:include filename="$(find premaidai_description)/urdf/arm.urdf.xacro" />
   <xacro:include filename="$(find premaidai_description)/urdf/body.urdf.xacro" />
   <link name="base_link"/>
-  <xacro:premaidai_rleg prefix="rleg" parent="base_link">
-    <origin xyz="0 0 0" rpy="0 0 0"/>
-  </xacro:premaidai_rleg>
-  <xacro:premaidai_lleg prefix="lleg" parent="base_link">
-    <origin xyz="0 0 0" rpy="0 0 0"/>
-  </xacro:premaidai_lleg>
-  <xacro:premaidai_rarm prefix="rarm" parent="base_link">
-    <origin xyz="0 0 0" rpy="0 0 0"/>
-  </xacro:premaidai_rarm>
-  <xacro:premaidai_larm prefix="larm" parent="base_link">
-    <origin xyz="0 0 0" rpy="0 0 0"/>
-  </xacro:premaidai_larm>
+  <xacro:premaidai_leg prefix="r" parent="base_link" sign="-1.0">
+    <origin xyz="0 -0.0217 0.01505" rpy="0 0 0"/>
+  </xacro:premaidai_leg>
+  <xacro:premaidai_leg prefix="l" parent="base_link" sign="1.0">
+    <origin xyz="0 0.0217 0.01505" rpy="0 0 0"/>
+  </xacro:premaidai_leg>
+  <xacro:premaidai_arm prefix="r" parent="base_link" sign="-1.0">
+    <origin xyz="-0.01726 -0.03829 0.097" rpy="0 0 0"/>
+  </xacro:premaidai_arm>
+  <xacro:premaidai_arm prefix="l" parent="base_link" sign="1.0">
+    <origin xyz="-0.01726 0.03829 0.097" rpy="0 0 0"/>
+  </xacro:premaidai_arm>
   <xacro:premaidai_body parent="base_link">
     <origin xyz="0 0 0" rpy="0 0 0"/>

File: urdf/arm.urdf.xacro (robot description, xacro)
@@ -1,34 +1,34 @@
 <?xml version="1.0"?>
 <robot name="arm" xmlns:xacro="http://ros.org/wiki/xacro">
-  <xacro:macro name="premaidai_rarm" params="prefix parent *origin">
-    <link name="${prefix}_1y">
+  <xacro:macro name="premaidai_arm" params="prefix parent sign *origin">
+    <link name="${prefix}_uarm_joint">
       <visual>
         <origin rpy="0 0 0" xyz="0 0 0"/>
         <geometry>
-          <mesh filename="package://premaidai_description/meshes/${prefix}_1y.dae"/>
+          <mesh filename="package://premaidai_description/meshes/${prefix}_uarm_joint.dae"/>
         </geometry>
       </visual>
     </link>
-    <link name="${prefix}_1x">
+    <link name="${prefix}_uarm">
       <visual>
         <origin rpy="0 0 0" xyz="0 0 0"/>
         <geometry>
-          <mesh filename="package://premaidai_description/meshes/${prefix}_1x.dae"/>
+          <mesh filename="package://premaidai_description/meshes/${prefix}_uarm.dae"/>
         </geometry>
       </visual>
     </link>
-    <link name="${prefix}_2z">
+    <link name="${prefix}_larm_joint">
       <visual>
         <origin rpy="0 0 0" xyz="0 0 0"/>
         <geometry>
-          <mesh filename="package://premaidai_description/meshes/${prefix}_2z.dae"/>
+          <mesh filename="package://premaidai_description/meshes/${prefix}_larm_joint.dae"/>
         </geometry>
       </visual>
     </link>
-    <link name="${prefix}_2x">
+    <link name="${prefix}_larm">
       <visual>
         <origin rpy="0 0 0" xyz="0 0 0"/>
         <geometry>
-          <mesh filename="package://premaidai_description/meshes/${prefix}_2x.dae"/>
+          <mesh filename="package://premaidai_description/meshes/${prefix}_larm.dae"/>
         </geometry>
       </visual>
@@ -43,36 +43,36 @@
     </link>
     <joint name="${prefix}_shy_joint" type="revolute">
-      <origin xyz="-0.01726 -0.03829 0.097" rpy="0 0 0"/>
+      <xacro:insert_block name="origin" />
       <axis xyz="0 1 0"/>
       <limit lower="${-pi/2.0}" upper="${pi/2.0}" effort="0" velocity="0"/>
       <parent link="${parent}"/>
-      <child link="${prefix}_1y"/>
+      <child link="${prefix}_uarm_joint"/>
     </joint>
     <joint name="${prefix}_shx_joint" type="revolute">
-      <origin xyz="0 -0.01925 0" rpy="0 0 0"/>
+      <origin xyz="0 ${sign*0.01925} 0" rpy="0 0 0"/>
       <axis xyz="1 0 0"/>
       <limit lower="${-pi/2.0}" upper="${pi/2.0}" effort="0" velocity="0"/>
-      <parent link="${prefix}_1y"/>
-      <child link="${prefix}_1x"/>
+      <parent link="${prefix}_uarm_joint"/>
+      <child link="${prefix}_uarm"/>
     </joint>
     <joint name="${prefix}_ely_joint" type="revolute">
-      <origin xyz="0 -0.05587567 0" rpy="0 0 0"/>
+      <origin xyz="0 ${sign*0.05587567} 0" rpy="0 0 0"/>
       <axis xyz="0 1 0"/>
       <limit lower="${-pi/2.0}" upper="${pi/2.0}" effort="0" velocity="0"/>
-      <parent link="${prefix}_1x"/>
-      <child link="${prefix}_2z"/>
+      <parent link="${prefix}_uarm"/>
+      <child link="${prefix}_larm_joint"/>
     </joint>
     <joint name="${prefix}_elx_joint" type="revolute">
-      <origin xyz="0 -0.030488976696505 0" rpy="0 0 0"/>
+      <origin xyz="0 ${sign*0.030488976696505} 0" rpy="0 0 0"/>
       <axis xyz="1 0 0"/>
       <limit lower="${-pi/2.0}" upper="${pi/2.0}" effort="0" velocity="0"/>
-      <parent link="${prefix}_2z"/>
-      <child link="${prefix}_2x"/>
+      <parent link="${prefix}_larm_joint"/>
+      <child link="${prefix}_larm"/>
     </joint>
     <joint name="${prefix}_wry_joint" type="revolute">
-      <origin xyz="0.01002 -0.047611784255581 0" rpy="0 0 0"/>
+      <origin xyz="0.01002 ${sign*0.047611784255581} 0" rpy="0 0 0"/>
       <axis xyz="0 1 0"/>
       <limit lower="${-pi/2.0}" upper="${pi/2.0}" effort="0" velocity="0"/>
-      <parent link="${prefix}_2x"/>
+      <parent link="${prefix}_larm"/>
       <child link="${prefix}_hand"/>
     </joint>

File: urdf/leg.urdf.xacro (robot description, xacro)
@@ -1,34 +1,34 @@
 <?xml version="1.0"?>
-<robot name="rleg" xmlns:xacro="http://ros.org/wiki/xacro">
-  <xacro:macro name="premaidai_rleg" params="prefix parent *origin">
-    <link name="${prefix}_1z">
+<robot name="leg" xmlns:xacro="http://ros.org/wiki/xacro">
+  <xacro:macro name="premaidai_leg" params="prefix parent sign *origin">
+    <link name="${prefix}_hip_joint">
       <visual>
         <origin rpy="0 0 0" xyz="0 0 0"/>
         <geometry>
-          <mesh filename="package://premaidai_description/meshes/${prefix}_1z.dae"/>
+          <mesh filename="package://premaidai_description/meshes/${prefix}_hip_joint.dae"/>
         </geometry>
       </visual>
     </link>
-    <link name="${prefix}_1y">
+    <link name="${prefix}_uleg_root">
       <visual>
         <origin rpy="0 0 0" xyz="0 0 0"/>
         <geometry>
-          <mesh filename="package://premaidai_description/meshes/${prefix}_1y.dae"/>
+          <mesh filename="package://premaidai_description/meshes/${prefix}_uleg_root.dae"/>
         </geometry>
       </visual>
     </link>
-    <link name="${prefix}_1x">
+    <link name="${prefix}_uleg">
       <visual>
         <origin rpy="0 0 0" xyz="0 0 0"/>
         <geometry>
-          <mesh filename="package://premaidai_description/meshes/${prefix}_1x.dae"/>
+          <mesh filename="package://premaidai_description/meshes/${prefix}_uleg.dae"/>
         </geometry>
       </visual>
     </link>
-    <link name="${prefix}_2y">
+    <link name="${prefix}_lleg">
       <visual>
         <origin rpy="0 0 0" xyz="0 0 0"/>
         <geometry>
-          <mesh filename="package://premaidai_description/meshes/${prefix}_2y.dae"/>
+          <mesh filename="package://premaidai_description/meshes/${prefix}_lleg.dae"/>
         </geometry>
       </visual>
@@ -51,9 +51,9 @@
     </link>
     <joint name="${prefix}_hpz_joint" type="revolute">
-      <origin xyz="0 -0.0217 0.01505" rpy="0 0 0"/>
+      <xacro:insert_block name="origin" />
       <axis xyz="0 0 1"/>
       <limit lower="${-pi/2.0}" upper="${pi/2.0}" effort="0" velocity="0"/>
       <parent link="${parent}"/>
-      <child link="${prefix}_1z"/>
+      <child link="${prefix}_hip_joint"/>
     </joint>
     <joint name="${prefix}_hpx_joint" type="revolute">
@@ -61,13 +61,13 @@
       <axis xyz="1 0 0"/>
       <limit lower="${-pi/2.0}" upper="${pi/2.0}" effort="0" velocity="0"/>
-      <parent link="${prefix}_1z"/>
-      <child link="${prefix}_1y"/>
+      <parent link="${prefix}_hip_joint"/>
+      <child link="${prefix}_uleg_root"/>
     </joint>
     <joint name="${prefix}_hpy_joint" type="revolute">
-      <origin xyz="0 -0.01021 -0.03829" rpy="0 0 0"/>
+      <origin xyz="0 ${sign*0.01021} -0.03829" rpy="0 0 0"/>
       <axis xyz="0 1 0"/>
       <limit lower="${-pi/2.0}" upper="${pi/2.0}" effort="0" velocity="0"/>
-      <parent link="${prefix}_1y"/>
-      <child link="${prefix}_1x"/>
+      <parent link="${prefix}_uleg_root"/>
+      <child link="${prefix}_uleg"/>
     </joint>
     <joint name="${prefix}_kny_joint" type="revolute">
@@ -75,11 +75,11 @@
       <axis xyz="0 1 0"/>
       <limit lower="${-pi/2.0}" upper="${pi/2.0}" effort="0" velocity="0"/>
-      <parent link="${prefix}_1x"/>
-      <child link="${prefix}_2y"/>
+      <parent link="${prefix}_uleg"/>
+      <child link="${prefix}_lleg"/>
     </joint>
     <joint name="${prefix}_aky_joint" type="revolute">
       <axis xyz="0 1 0"/>
       <limit lower="${-pi/2.0}" upper="${pi/2.0}" effort="0" velocity="0"/>
-      <parent link="${prefix}_2y"/>
+      <parent link="${prefix}_lleg"/>
       <child link="${prefix}_dummy"/>
     </joint>
