Commit message: Update model

File: robots/premaidai.urdf.xacro (robot description, xacro)
@@ -8,14 +8,14 @@
   <link name="base_link"/>
   <xacro:premaidai_leg prefix="r" parent="base_link" sign="-1.0">
-    <origin xyz="0 -0.0217 0.01505" rpy="0 0 0"/>
+    <origin xyz="0.004225 -0.0195245 0.001412" rpy="0 0 0"/>
   </xacro:premaidai_leg>
   <xacro:premaidai_leg prefix="l" parent="base_link" sign="1.0">
-    <origin xyz="0 0.0217 0.01505" rpy="0 0 0"/>
+    <origin xyz="0.004225 0.0195245 0.001412" rpy="0 0 0"/>
   </xacro:premaidai_leg>
   <xacro:premaidai_arm prefix="r" parent="base_link" sign="-1.0">
-    <origin xyz="-0.01726 -0.03829 0.097" rpy="0 0 0"/>
+    <origin xyz="0 -0.0359 0.113043" rpy="0 0 0"/>
   </xacro:premaidai_arm>
   <xacro:premaidai_arm prefix="l" parent="base_link" sign="1.0">
-    <origin xyz="-0.01726 0.03829 0.097" rpy="0 0 0"/>
+    <origin xyz="0 0.0359 0.113043" rpy="0 0 0"/>
   </xacro:premaidai_arm>
   <xacro:premaidai_body parent="base_link">

File: urdf/arm.urdf.xacro (robot description, xacro)
@@ -6,5 +6,5 @@
         <origin rpy="0 0 0" xyz="0 0 0"/>
         <geometry>
-          <mesh filename="package://premaidai_description/meshes/${prefix}_uarm_joint.dae"/>
+          <mesh filename="package://premaidai_description/meshes/${prefix}_uarm_joint.dae" scale="0.01 0.01 0.01"/>
         </geometry>
       </visual>
@@ -12,5 +12,5 @@
         <origin rpy="0 0 0" xyz="0 0 0"/>
         <geometry>
-          <mesh filename="package://premaidai_description/meshes/${prefix}_uarm_joint.dae"/>
+          <mesh filename="package://premaidai_description/meshes/${prefix}_uarm_joint.dae" scale="0.01 0.01 0.01"/>
         </geometry>
       </collision>
@@ -20,5 +20,5 @@
         <origin rpy="0 0 0" xyz="0 0 0"/>
         <geometry>
-          <mesh filename="package://premaidai_description/meshes/${prefix}_uarm.dae"/>
+          <mesh filename="package://premaidai_description/meshes/${prefix}_uarm.dae" scale="0.01 0.01 0.01"/>
         </geometry>
       </visual>
@@ -26,5 +26,5 @@
         <origin rpy="0 0 0" xyz="0 0 0"/>
         <geometry>
-          <mesh filename="package://premaidai_description/meshes/${prefix}_uarm.dae"/>
+          <mesh filename="package://premaidai_description/meshes/${prefix}_uarm.dae" scale="0.01 0.01 0.01"/>
         </geometry>
       </collision>
@@ -34,5 +34,5 @@
         <origin rpy="0 0 0" xyz="0 0 0"/>
         <geometry>
-          <mesh filename="package://premaidai_description/meshes/${prefix}_larm_joint.dae"/>
+          <mesh filename="package://premaidai_description/meshes/${prefix}_larm_joint.dae" scale="0.01 0.01 0.01"/>
         </geometry>
       </visual>
@@ -40,5 +40,5 @@
         <origin rpy="0 0 0" xyz="0 0 0"/>
         <geometry>
-          <mesh filename="package://premaidai_description/meshes/${prefix}_larm_joint.dae"/>
+          <mesh filename="package://premaidai_description/meshes/${prefix}_larm_joint.dae" scale="0.01 0.01 0.01"/>
         </geometry>
       </collision>
@@ -48,5 +48,5 @@
         <origin rpy="0 0 0" xyz="0 0 0"/>
         <geometry>
-          <mesh filename="package://premaidai_description/meshes/${prefix}_larm.dae"/>
+          <mesh filename="package://premaidai_description/meshes/${prefix}_larm.dae" scale="0.01 0.01 0.01"/>
         </geometry>
       </visual>
@@ -54,5 +54,5 @@
         <origin rpy="0 0 0" xyz="0 0 0"/>
         <geometry>
-          <mesh filename="package://premaidai_description/meshes/${prefix}_larm.dae"/>
+          <mesh filename="package://premaidai_description/meshes/${prefix}_larm.dae" scale="0.01 0.01 0.01"/>
         </geometry>
       </collision>
@@ -62,5 +62,5 @@
         <origin rpy="0 0 0" xyz="0 0 0"/>
         <geometry>
-          <mesh filename="package://premaidai_description/meshes/${prefix}_hand.dae"/>
+          <mesh filename="package://premaidai_description/meshes/${prefix}_hand.dae" scale="0.01 0.01 0.01"/>
         </geometry>
       </visual>
@@ -68,5 +68,5 @@
         <origin rpy="0 0 0" xyz="0 0 0"/>
         <geometry>
-          <mesh filename="package://premaidai_description/meshes/${prefix}_hand.dae"/>
+          <mesh filename="package://premaidai_description/meshes/${prefix}_hand.dae" scale="0.01 0.01 0.01"/>
         </geometry>
       </collision>
@@ -80,12 +80,12 @@
     </joint>
     <joint name="${prefix}_shx_joint" type="revolute">
-      <origin xyz="0 ${sign*0.01925} 0" rpy="0 0 0"/>
+      <origin xyz="0 ${sign*0.0189} 0" rpy="0 0 0"/>
       <axis xyz="1 0 0"/>
-      <limit lower="${-pi/2.0}" upper="${pi/2.0}" effort="0" velocity="0"/>
+      <limit lower="${-pi / 2.0}" upper="${pi / 2.0}" effort="0" velocity="0"/>
       <parent link="${prefix}_uarm_joint"/>
       <child link="${prefix}_uarm"/>
     </joint>
     <joint name="${prefix}_ely_joint" type="revolute">
-      <origin xyz="0 ${sign*0.05587567} 0" rpy="0 0 0"/>
+      <origin xyz="0.0088013 ${sign*0.060007} 0" rpy="0 0 0"/>
       <axis xyz="0 1 0"/>
       <limit lower="${-pi/2.0}" upper="${pi/2.0}" effort="0" velocity="0"/>
@@ -94,5 +94,5 @@
     </joint>
     <joint name="${prefix}_elx_joint" type="revolute">
-      <origin xyz="0 ${sign*0.030488976696505} 0" rpy="0 0 0"/>
+      <origin xyz="0 ${sign*0.024054} 0" rpy="0 0 0"/>
       <axis xyz="1 0 0"/>
       <limit lower="${-pi/2.0}" upper="${pi/2.0}" effort="0" velocity="0"/>
@@ -101,5 +101,5 @@
     </joint>
     <joint name="${prefix}_wry_joint" type="revolute">
-      <origin xyz="0.01002 ${sign*0.047611784255581} 0" rpy="0 0 0"/>
+      <origin xyz="0 ${sign*0.061348} 0" rpy="0 0 0"/>
       <axis xyz="0 1 0"/>
       <limit lower="${-pi/2.0}" upper="${pi/2.0}" effort="0" velocity="0"/>

File: urdf/body.urdf.xacro (robot description, xacro)
@@ -5,79 +5,75 @@
       <visual>
         <geometry>
-            <mesh filename="package://premaidai_description/meshes/body.dae"/>
+          <mesh filename="package://premaidai_description/meshes/body.dae" scale="0.01 0.01 0.01"/>
         </geometry>
       </visual>
       <collision>
         <geometry>
-            <mesh filename="package://premaidai_description/meshes/body.dae"/>
+          <mesh filename="package://premaidai_description/meshes/body.dae" scale="0.01 0.01 0.01"/>
         </geometry>
       </collision>
     </link>
-    <link name="neck">
+    <link name="neck_pitch">
       <visual>
         <geometry>
-            <mesh filename="package://premaidai_description/meshes/neck.dae"/>
+          <mesh filename="package://premaidai_description/meshes/neck_pitch.dae" scale="0.01 0.01 0.01"/>
         </geometry>
       </visual>
       <collision>
         <geometry>
-            <mesh filename="package://premaidai_description/meshes/neck.dae"/>
+          <mesh filename="package://premaidai_description/meshes/neck_pitch.dae" scale="0.01 0.01 0.01"/>
         </geometry>
       </collision>
     </link>
-    <link name="head_dummy">
+    <link name="head_yaw">
       <visual>
         <geometry>
-          <box size="0.01 0.01 0.01" />
+          <mesh filename="package://premaidai_description/meshes/neck_yaw.dae" scale="0.01 0.01 0.01"/>
         </geometry>
       </visual>
+      <collision>
+        <geometry>
+          <mesh filename="package://premaidai_description/meshes/neck_yaw.dae" scale="0.01 0.01 0.01"/>
+        </geometry>
+      </collision>
     </link>
     <link name="head">
       <visual>
         <geometry>
-            <mesh filename="package://premaidai_description/meshes/head.dae"/>
+          <mesh filename="package://premaidai_description/meshes/head.dae" scale="0.01 0.01 0.01"/>
         </geometry>
       </visual>
       <collision>
         <geometry>
-            <mesh filename="package://premaidai_description/meshes/head.dae"/>
+          <mesh filename="package://premaidai_description/meshes/head.dae" scale="0.01 0.01 0.01"/>
         </geometry>
       </collision>
     </link>
     <joint name="body_to_base_link" type="fixed">
-      <origin xyz="0.0236 0 0" rpy="0 0 0"/>
+      <origin xyz="0 0 0" rpy="0 0 0"/>
       <parent link="${parent}"/>
       <child link="body"/>
     </joint>
     <joint name="head_ny_joint" type="revolute">
-      <origin xyz="-0.0319 0 0.1088" rpy="0 0 0"/>
+      <origin xyz="0.0038738 0 0.132809" rpy="0 0 0"/>
       <axis xyz="0 1 0"/>
       <limit lower="${-10.125/180.0 * pi}" upper="${23.625/180.0 * pi}" effort="0" velocity="0"/>
       <parent link="body"/>
-      <child link="neck"/>
+      <child link="neck_pitch"/>
     </joint>
     <joint name="head_nz_joint" type="revolute">
-      <origin xyz="0 0 0" rpy="0 0 0"/>
+      <origin xyz="-0.0103485 0 0.011103" rpy="0 0 0"/>
       <axis xyz="0 0 1"/>
       <limit lower="${-47.25/180.0 * pi}" upper="${47.25/180.0 * pi}" effort="0" velocity="0"/>
-      <parent link="neck"/>
-      <child link="head_dummy"/>
+      <parent link="neck_pitch"/>
+      <child link="head_yaw"/>
     </joint>
     <joint name="head_nx_joint" type="revolute">
-      <origin xyz="0 0 0.0362" rpy="0 0 0"/>
+      <origin xyz="0 0 0.0129" rpy="0 0 0"/>
       <axis xyz="1 0 0"/>
       <limit lower="${-21.9375/180.0 * pi}" upper="${28.6875/180.0 * pi}" effort="0" velocity="0"/>
-      <parent link="head_dummy"/>
+      <parent link="head_yaw"/>
       <child link="head"/>
     </joint>
-<!-- MUST implement
-    <joint name="head_yaw_joint" type="revolute">
-      <origin xyz="0 0 0.0362" rpy="0 0 0"/>
-      <axis xyz="0 1 0"/>
-      <limit lower="0" upper="0" effort="0" velocity="0"/>
-      <parent link="neck"/>
-      <child link="head"/>
-    </joint>
- -->
   </xacro:macro>
 </robot>

File: urdf/leg.urdf.xacro (robot description, xacro)
@@ -6,5 +6,5 @@
         <origin rpy="0 0 0" xyz="0 0 0"/>
         <geometry>
-          <mesh filename="package://premaidai_description/meshes/${prefix}_hip_joint.dae"/>
+          <mesh filename="package://premaidai_description/meshes/${prefix}_hip_joint.dae" scale="0.01 0.01 0.01"/>
         </geometry>
       </visual>
@@ -12,5 +12,5 @@
         <origin rpy="0 0 0" xyz="0 0 0"/>
         <geometry>
-          <mesh filename="package://premaidai_description/meshes/${prefix}_hip_joint.dae"/>
+          <mesh filename="package://premaidai_description/meshes/${prefix}_hip_joint.dae" scale="0.01 0.01 0.01"/>
         </geometry>
       </collision>
@@ -20,5 +20,5 @@
         <origin rpy="0 0 0" xyz="0 0 0"/>
         <geometry>
-          <mesh filename="package://premaidai_description/meshes/${prefix}_uleg_root.dae"/>
+          <mesh filename="package://premaidai_description/meshes/${prefix}_uleg_root.dae" scale="0.01 0.01 0.01"/>
         </geometry>
       </visual>
@@ -26,5 +26,5 @@
         <origin rpy="0 0 0" xyz="0 0 0"/>
         <geometry>
-          <mesh filename="package://premaidai_description/meshes/${prefix}_uleg_root.dae"/>
+          <mesh filename="package://premaidai_description/meshes/${prefix}_uleg_root.dae" scale="0.01 0.01 0.01"/>
         </geometry>
       </collision>
@@ -34,5 +34,5 @@
         <origin rpy="0 0 0" xyz="0 0 0"/>
         <geometry>
-          <mesh filename="package://premaidai_description/meshes/${prefix}_uleg.dae"/>
+          <mesh filename="package://premaidai_description/meshes/${prefix}_uleg.dae" scale="0.01 0.01 0.01"/>
         </geometry>
       </visual>
@@ -40,5 +40,5 @@
         <origin rpy="0 0 0" xyz="0 0 0"/>
         <geometry>
-          <mesh filename="package://premaidai_description/meshes/${prefix}_uleg.dae"/>
+          <mesh filename="package://premaidai_description/meshes/${prefix}_uleg.dae" scale="0.01 0.01 0.01"/>
         </geometry>
       </collision>
@@ -48,5 +48,5 @@
         <origin rpy="0 0 0" xyz="0 0 0"/>
         <geometry>
-          <mesh filename="package://premaidai_description/meshes/${prefix}_lleg.dae"/>
+          <mesh filename="package://premaidai_description/meshes/${prefix}_lleg.dae" scale="0.01 0.01 0.01"/>
         </geometry>
       </visual>
@@ -54,15 +54,21 @@
         <origin rpy="0 0 0" xyz="0 0 0"/>
         <geometry>
-          <mesh filename="package://premaidai_description/meshes/${prefix}_lleg.dae"/>
+          <mesh filename="package://premaidai_description/meshes/${prefix}_lleg.dae" scale="0.01 0.01 0.01"/>
         </geometry>
       </collision>
     </link>
-    <link name="${prefix}_dummy">
+    <link name="${prefix}_ankle">
       <visual>
         <origin rpy="0 0 0" xyz="0 0 0"/>
         <geometry>
-          <box size="0.01 0.01 0.01" />
+          <mesh filename="package://premaidai_description/meshes/${prefix}_ankle.dae" scale="0.01 0.01 0.01"/>
         </geometry>
       </visual>
+      <collision>
+        <origin rpy="0 0 0" xyz="0 0 0"/>
+        <geometry>
+          <mesh filename="package://premaidai_description/meshes/${prefix}_ankle.dae" scale="0.01 0.01 0.01"/>
+        </geometry>
+      </collision>
     </link>
     <link name="${prefix}_foot">
@@ -70,5 +76,5 @@
         <origin rpy="0 0 0" xyz="0 0 0"/>
         <geometry>
-          <mesh filename="package://premaidai_description/meshes/${prefix}_foot.dae"/>
+          <mesh filename="package://premaidai_description/meshes/${prefix}_foot.dae" scale="0.01 0.01 0.01"/>
         </geometry>
       </visual>
@@ -76,5 +82,5 @@
         <origin rpy="0 0 0" xyz="0 0 0"/>
         <geometry>
-          <mesh filename="package://premaidai_description/meshes/${prefix}_foot.dae"/>
+          <mesh filename="package://premaidai_description/meshes/${prefix}_foot.dae" scale="0.01 0.01 0.01"/>
         </geometry>
       </collision>
@@ -88,5 +94,5 @@
     </joint>
     <joint name="${prefix}_hpx_joint" type="revolute">
-      <origin xyz="0 0 -0.05407" rpy="0 0 0"/>
+      <origin xyz="0 ${sign*-0.0021} -0.028" rpy="0 0 0"/>
       <axis xyz="1 0 0"/>
       <limit lower="${-pi/2.0}" upper="${pi/2.0}" effort="0" velocity="0"/>
@@ -95,5 +101,5 @@
     </joint>
     <joint name="${prefix}_hpy_joint" type="revolute">
-      <origin xyz="0 ${sign*0.01021} -0.03829" rpy="0 0 0"/>
+      <origin xyz="0 ${sign*0.0128525} -0.034358" rpy="0 0 0"/>
       <axis xyz="0 1 0"/>
       <limit lower="${-pi/2.0}" upper="${pi/2.0}" effort="0" velocity="0"/>
@@ -102,5 +108,5 @@
     </joint>
     <joint name="${prefix}_kny_joint" type="revolute">
-      <origin xyz="0 0 -0.06827" rpy="0 0 0"/>
+      <origin xyz="0 0 -0.0652" rpy="0 0 0"/>
       <axis xyz="0 1 0"/>
       <limit lower="${-pi/2.0}" upper="${pi/2.0}" effort="0" velocity="0"/>
@@ -109,14 +115,15 @@
     </joint>
     <joint name="${prefix}_aky_joint" type="revolute">
-      <origin xyz="0 0 -0.06749" rpy="0 0 0"/>
+      <origin xyz="0 0 -0.065" rpy="0 0 0"/>
       <axis xyz="0 1 0"/>
       <limit lower="${-pi/2.0}" upper="${pi/2.0}" effort="0" velocity="0"/>
       <parent link="${prefix}_lleg"/>
-      <child link="${prefix}_dummy"/>
+      <child link="${prefix}_ankle"/>
     </joint>
     <joint name="${prefix}_akx_joint" type="revolute">
+      <origin xyz="0 0 -0.040677" rpy="0 0 0"/>
       <axis xyz="1 0 0"/>
       <limit lower="${-pi/2.0}" upper="${pi/2.0}" effort="0" velocity="0"/>
-      <parent link="${prefix}_dummy"/>
+      <parent link="${prefix}_ankle"/>
       <child link="${prefix}_foot"/>
     </joint>

Commit message: Add right/left definition macro to xacro files

File: robots/premaidai.urdf.xacro (robot description, xacro)
@@ -7,14 +7,14 @@
   <xacro:include filename="$(find premaidai_description)/urdf/body.urdf.xacro" />
   <link name="base_link"/>
-  <xacro:premaidai_leg prefix="r" parent="base_link" sign="-1.0">
+  <xacro:premaidai_leg prefix="r" parent="base_link" side="right">
     <origin xyz="0.004225 -0.0195245 0.001412" rpy="0 0 0"/>
   </xacro:premaidai_leg>
-  <xacro:premaidai_leg prefix="l" parent="base_link" sign="1.0">
+  <xacro:premaidai_leg prefix="l" parent="base_link" side="left">
     <origin xyz="0.004225 0.0195245 0.001412" rpy="0 0 0"/>
   </xacro:premaidai_leg>
-  <xacro:premaidai_arm prefix="r" parent="base_link" sign="-1.0">
+  <xacro:premaidai_arm prefix="r" parent="base_link" side="right">
     <origin xyz="0 -0.0359 0.113043" rpy="0 0 0"/>
   </xacro:premaidai_arm>
-  <xacro:premaidai_arm prefix="l" parent="base_link" sign="1.0">
+  <xacro:premaidai_arm prefix="l" parent="base_link" side="left">
     <origin xyz="0 0.0359 0.113043" rpy="0 0 0"/>
   </xacro:premaidai_arm>

File: urdf/arm.urdf.xacro (robot description, xacro)
@@ -1,5 +1,11 @@
 <?xml version="1.0"?>
 <robot name="arm" xmlns:xacro="http://ros.org/wiki/xacro">
-  <xacro:macro name="premaidai_arm" params="prefix parent sign *origin">
+  <xacro:macro name="premaidai_arm" params="prefix parent side *origin">
+    <xacro:if value="${side=='right'}">
+      <xacro:property name="sign" value="-1"/>
+    </xacro:if>
+    <xacro:if value="${side=='left'}">
+      <xacro:property name="sign" value="1"/>
+    </xacro:if>
     <link name="${prefix}_uarm_joint">
       <visual>

File: urdf/leg.urdf.xacro (robot description, xacro)
@@ -1,5 +1,11 @@
 <?xml version="1.0"?>
 <robot name="leg" xmlns:xacro="http://ros.org/wiki/xacro">
-  <xacro:macro name="premaidai_leg" params="prefix parent sign *origin">
+  <xacro:macro name="premaidai_leg" params="prefix parent side *origin">
+    <xacro:if value="${side=='right'}">
+      <xacro:property name="sign" value="-1"/>
+    </xacro:if>
+    <xacro:if value="${side=='left'}">
+      <xacro:property name="sign" value="1"/>
+    </xacro:if>
     <link name="${prefix}_hip_joint">
       <visual>
