Commit message: Add inertia parameters to urdf

File: robots/premaidai.urdf.xacro (robot description, xacro)
@@ -4,21 +4,29 @@
   <xacro:include filename="$(find premaidai_description)/urdf/common.xacro" />
   <xacro:include filename="$(find premaidai_description)/urdf/leg.urdf.xacro" />
+  <xacro:include filename="$(find premaidai_description)/urdf/leg.gazebo.xacro" />
   <xacro:include filename="$(find premaidai_description)/urdf/arm.urdf.xacro" />
+  <xacro:include filename="$(find premaidai_description)/urdf/arm.gazebo.xacro" />
   <xacro:include filename="$(find premaidai_description)/urdf/body.urdf.xacro" />
+  <xacro:include filename="$(find premaidai_description)/urdf/body.gazebo.xacro" />
   <link name="base_link"/>
   <xacro:premaidai_leg prefix="r" parent="base_link" side="right">
     <origin xyz="0.004225 -0.0195245 0.001412" rpy="0 0 0"/>
   </xacro:premaidai_leg>
+  <xacro:premaidai_leg_gazebo prefix="r"/>
   <xacro:premaidai_leg prefix="l" parent="base_link" side="left">
     <origin xyz="0.004225 0.0195245 0.001412" rpy="0 0 0"/>
   </xacro:premaidai_leg>
+  <xacro:premaidai_leg_gazebo prefix="l"/>
   <xacro:premaidai_arm prefix="r" parent="base_link" side="right">
     <origin xyz="0 -0.0359 0.113043" rpy="0 0 0"/>
   </xacro:premaidai_arm>
+  <xacro:premaidai_arm_gazebo prefix="r"/>
   <xacro:premaidai_arm prefix="l" parent="base_link" side="left">
     <origin xyz="0 0.0359 0.113043" rpy="0 0 0"/>
   </xacro:premaidai_arm>
+  <xacro:premaidai_arm_gazebo prefix="l"/>
   <xacro:premaidai_body parent="base_link">
     <origin xyz="0 0 0" rpy="0 0 0"/>
   </xacro:premaidai_body>
+  <xacro:premaidai_body_gazebo/>
 </robot>

File: urdf/arm.urdf.xacro (robot description, xacro)
@@ -21,4 +21,9 @@
         </geometry>
       </collision>
+      <inertial>
+        <mass value="0.0131"/>
+        <origin xyz="-0.000000 ${sign*0.005109} 0.000865"/>
+        <inertia ixx="39.090332e-10" ixy="0.000021e-10" ixz="0.000003e-10" iyy="116.438423e-10" iyz="${sign*-4.044059e-10}" izz="132.243393e-10"/>
+      </inertial>
     </link>
     <link name="${prefix}_uarm">
@@ -35,4 +40,9 @@
         </geometry>
       </collision>
+      <inertial>
+        <mass value="0.0712"/>
+        <origin xyz="-0.000001 ${sign*0.021640} 0.000670"/>
+        <inertia ixx="356.620514e-10" ixy="-0.000020e-10" ixz="0.000026e-10" iyy="126.890160e-10" iyz="${sign*4.816492e-10}" izz="414.000244e-10"/>
+      </inertial>
     </link>
     <link name="${prefix}_larm_joint">
@@ -49,4 +59,9 @@
         </geometry>
       </collision>
+      <inertial>
+        <mass value="0.0124"/>
+        <origin xyz="-0.008596 ${sign*0.015762} 0.002150"/>
+        <inertia ixx="70.485497e-10" ixy="${sign*104.342163e-10}" ixz="-0.000005e-10" iyy="188.648819e-10" iyz="${sign*-3.846500e-10}" izz="236.494141e-10"/>
+      </inertial>
     </link>
     <link name="${prefix}_larm">
@@ -63,4 +78,9 @@
         </geometry>
       </collision>
+      <inertial>
+        <mass value="0.0812"/>
+        <origin xyz="-0.008596 ${sign*0.027572} 0.000420"/>
+        <inertia ixx="342.361237e-10" ixy="${sign*-0.000036e-10}" ixz="0.000012e-10" iyy="141.587677e-10" iyz="${sign*0.382193e-10}" izz="414.116486e-10"/>
+      </inertial>
     </link>
     <link name="${prefix}_hand">
@@ -77,4 +97,9 @@
         </geometry>
       </collision>
+      <inertial>
+        <mass value="0.0046"/>
+        <origin xyz="0.001817 ${sign*0.018911} 0.002717"/>
+        <inertia ixx="8.193970e-10" ixy="${sign*-0.178483e-10}" ixz="0.194812e-10" iyy="3.111708e-10" iyz="${sign*-2.003531e-10}" izz="9.081884e-10"/>
+      </inertial>
     </link>
     <joint name="${prefix}_shy_joint" type="revolute">

File: urdf/body.urdf.xacro (robot description, xacro)
@@ -13,4 +13,9 @@
         </geometry>
       </collision>
+      <inertial>
+        <mass value="0.4426"/>
+        <origin xyz="0.008509 0.000002 0.070698"/>
+        <inertia ixx="2871.143311e-10" ixy="-0.001151e-10" ixz="237.094467e-10" iyy="2672.078857e-10" iyz="-0.003379e-10" izz="1188.332153e-10"/>
+      </inertial>
     </link>
     <link name="neck_pitch">
@@ -25,4 +30,9 @@
         </geometry>
       </collision>
+      <inertial>
+        <mass value="0.01"/>
+        <origin xyz="-0.006449 0.000002 0.008964"/>
+        <inertia ixx="6.489763e-10" ixy="-0.000003e-10" ixz="-0.024047e-10" iyy="2.296302e-10" iyz="-0.000005e-10" izz="6.197822e-10"/>
+      </inertial>
     </link>
     <link name="head_yaw">
@@ -37,4 +47,9 @@
         </geometry>
       </collision>
+      <inertial>
+        <mass value="0.01"/>
+        <origin xyz="0.008100 0.000002 0.017871"/>
+        <inertia ixx="12.636111e-10" ixy="-0.000001e-10" ixz="0.0" iyy="23.689224e-10" iyz="0.0" izz="17.372910e-10"/>
+      </inertial>
     </link>
     <link name="head">
@@ -49,4 +64,9 @@
         </geometry>
       </collision>
+      <inertial>
+        <mass value="0.1449"/>
+        <origin xyz="0.014213 0.000001 0.011813"/>
+        <inertia ixx="650.041687e-10" ixy="-0.000280e-10" ixz="49.702934e-10" iyy="598.413635e-10" iyz="-0.000379e-10" izz="588.398682e-10"/>
+      </inertial>
     </link>
     <joint name="body_to_base_link" type="fixed">

File: urdf/leg.urdf.xacro (robot description, xacro)
@@ -21,4 +21,9 @@
         </geometry>
       </collision>
+      <inertial>
+        <mass value="0.0143"/>
+        <origin xyz="0.000000 ${sign*0.000183} -0.010532"/>
+        <inertia ixx="20.138887e-10" ixy="-0.000001e-10" ixz="0.0e-10" iyy="53.757824e-10" iyz="${sign*-0.518773e-10}" izz="46.127151e-10"/>
+      </inertial>
     </link>
     <link name="${prefix}_uleg_root">
@@ -35,4 +40,9 @@
         </geometry>
       </collision>
+      <inertial>
+        <mass value="0.0648"/>
+        <origin xyz="-0.000000 ${sign*0.013420} -0.004373"/>
+        <inertia ixx="246.003845e-10" ixy="${sign*-0.001517e-10}" ixz="-0.001688e-10" iyy="191.922195e-10" iyz="${sign*-6.165664e-10}" izz="238.454895e-10"/>
+      </inertial>
     </link>
     <link name="${prefix}_uleg">
@@ -49,4 +59,9 @@
         </geometry>
       </collision>
+      <inertial>
+        <mass value="0.1134"/>
+        <origin xyz="-0.000000 0.000001 -0.032601"/>
+        <inertia ixx="884.390869e-10" ixy="0.000002e-10" ixz="-0.000046e-10" iyy="825.489990e-10" iyz="-0.000031e-10" izz="222.801773e-10"/>
+      </inertial>
     </link>
     <link name="${prefix}_lleg">
@@ -63,4 +78,9 @@
         </geometry>
       </collision>
+      <inertial>
+        <mass value="0.0719"/>
+        <origin xyz="-0.001624 ${sign*0.002494} -0.034776"/>
+        <inertia ixx="735.568420e-10" ixy="${sign*-1.871153e-10}" ixz="-35.647034e-10" iyy="434.662354e-10" iyz="${sign*0.247592e-10}" izz="480.555054e-10"/>
+      </inertial>
     </link>
     <link name="${prefix}_ankle">
@@ -77,4 +97,9 @@
         </geometry>
       </collision>
+      <inertial>
+        <mass value="0.0571"/>
+        <origin xyz="-0.009629 0.000379 -0.003702"/>
+        <inertia ixx="175.244446e-10" ixy="-0.000004e-10" ixz="11.289989e-10" iyy="257.425598e-10" iyz="-0.000002e-10" izz="224.547821e-10"/>
+      </inertial>
     </link>
     <link name="${prefix}_foot">
@@ -91,4 +116,9 @@
         </geometry>
       </collision>
+      <inertial>
+        <mass value="0.0941"/>
+        <origin xyz="0.005014 ${sign*0.008793} -0.004123"/>
+        <inertia ixx="383.406982e-10" ixy="${sign*11.222215e-10}" ixz="12.157411e-10" iyy="1013.430359e-10" iyz="${sign*-1.649494e-10}" izz="1206.411377e-10"/>
+      </inertial>
     </link>
     <joint name="${prefix}_hpz_joint" type="revolute">
