Commit message: Fix inertia values

File: robots/premaidai.urdf.xacro (robot description, xacro)
@@ -30,3 +30,6 @@
   </xacro:premaidai_body>
   <xacro:premaidai_body_gazebo/>
+  <gazebo>
+    <plugin name="premaidai_plugin" filename="libPremaidAIPlugin.so"/>
+  </gazebo>
 </robot>

File: urdf/arm.gazebo.xacro (robot description, xacro)
@@ -3,17 +3,42 @@
   <xacro:macro name="premaidai_arm_gazebo" params="prefix">
     <gazebo reference="${prefix}_uarm_joint">
-      <selfCollide>true</selfCollide>
+      <!-- <selfCollide>false</selfCollide> -->
+      <mu1>0.9</mu1>
+      <mu2>0.9</mu2>
     </gazebo>
     <gazebo reference="${prefix}_uarm">
-      <selfCollide>true</selfCollide>
+      <!-- <selfCollide>false</selfCollide> -->
+      <mu1>0.9</mu1>
+      <mu2>0.9</mu2>
     </gazebo>
     <gazebo reference="${prefix}_larm_joint">
-      <selfCollide>true</selfCollide>
+      <!-- <selfCollide>false</selfCollide> -->
+      <mu1>0.9</mu1>
+      <mu2>0.9</mu2>
     </gazebo>
     <gazebo reference="${prefix}_larm">
-      <selfCollide>true</selfCollide>
+      <!-- <selfCollide>false</selfCollide> -->
+      <mu1>0.9</mu1>
+      <mu2>0.9</mu2>
     </gazebo>
     <gazebo reference="${prefix}_hand">
-      <selfCollide>true</selfCollide>
+      <!-- <selfCollide>false</selfCollide> -->
+      <mu1>0.9</mu1>
+      <mu2>0.9</mu2>
+    </gazebo>
+    <gazebo reference="${prefix}_shy_joint">
+      <implicitSpringDamper>1</implicitSpringDamper>
+    </gazebo>
+    <gazebo reference="${prefix}_shx_joint">
+      <implicitSpringDamper>1</implicitSpringDamper>
+    </gazebo>
+    <gazebo reference="${prefix}_ely_joint">
+      <implicitSpringDamper>1</implicitSpringDamper>
+    </gazebo>
+    <gazebo reference="${prefix}_elx_joint">
+      <implicitSpringDamper>1</implicitSpringDamper>
+    </gazebo>
+    <gazebo reference="${prefix}_wry_joint">
+      <implicitSpringDamper>1</implicitSpringDamper>
     </gazebo>
   </xacro:macro>

File: urdf/arm.urdf.xacro (robot description, xacro)
@@ -24,5 +24,5 @@
         <mass value="0.0131"/>
         <origin xyz="-0.000000 ${sign*0.005109} 0.000865"/>
-        <inertia ixx="39.090332e-10" ixy="0.000021e-10" ixz="0.000003e-10" iyy="116.438423e-10" iyz="${sign*-4.044059e-10}" izz="132.243393e-10"/>
+        <inertia ixx="39.090332e-5" ixy="0.000021e-5" ixz="0.000003e-5" iyy="116.438423e-5" iyz="${sign*-4.044059e-5}" izz="132.243393e-5"/>
       </inertial>
     </link>
@@ -43,5 +43,5 @@
         <mass value="0.0712"/>
         <origin xyz="-0.000001 ${sign*0.021640} 0.000670"/>
-        <inertia ixx="356.620514e-10" ixy="-0.000020e-10" ixz="0.000026e-10" iyy="126.890160e-10" iyz="${sign*4.816492e-10}" izz="414.000244e-10"/>
+        <inertia ixx="356.620514e-5" ixy="-0.000020e-5" ixz="0.000026e-5" iyy="126.890160e-5" iyz="${sign*4.816492e-5}" izz="414.000244e-5"/>
       </inertial>
     </link>
@@ -62,5 +62,5 @@
         <mass value="0.0124"/>
         <origin xyz="-0.008596 ${sign*0.015762} 0.002150"/>
-        <inertia ixx="70.485497e-10" ixy="${sign*104.342163e-10}" ixz="-0.000005e-10" iyy="188.648819e-10" iyz="${sign*-3.846500e-10}" izz="236.494141e-10"/>
+        <inertia ixx="70.485497e-5" ixy="${sign*104.342163e-5}" ixz="-0.000005e-5" iyy="188.648819e-5" iyz="${sign*-3.846500e-5}" izz="236.494141e-5"/>
       </inertial>
     </link>
@@ -81,5 +81,5 @@
         <mass value="0.0812"/>
         <origin xyz="-0.008596 ${sign*0.027572} 0.000420"/>
-        <inertia ixx="342.361237e-10" ixy="${sign*-0.000036e-10}" ixz="0.000012e-10" iyy="141.587677e-10" iyz="${sign*0.382193e-10}" izz="414.116486e-10"/>
+        <inertia ixx="342.361237e-5" ixy="${sign*-0.000036e-5}" ixz="0.000012e-5" iyy="141.587677e-5" iyz="${sign*0.382193e-5}" izz="414.116486e-5"/>
       </inertial>
     </link>
@@ -100,11 +100,19 @@
         <mass value="0.0046"/>
         <origin xyz="0.001817 ${sign*0.018911} 0.002717"/>
-        <inertia ixx="8.193970e-10" ixy="${sign*-0.178483e-10}" ixz="0.194812e-10" iyy="3.111708e-10" iyz="${sign*-2.003531e-10}" izz="9.081884e-10"/>
+        <inertia ixx="8.193970e-5" ixy="${sign*-0.178483e-5}" ixz="0.194812e-5" iyy="3.111708e-5" iyz="${sign*-2.003531e-5}" izz="9.081884e-5"/>
       </inertial>
+    </link>
+    <link name="${prefix}_hand_ee">
+      <collision>
+        <geometry>
+          <box size="0.01 0.01 0.01"/>
+        </geometry>
+        <origin rpy="0 0 0" xyz="-0.01 0 0"/>
+      </collision>
     </link>
     <joint name="${prefix}_shy_joint" type="revolute">
       <xacro:insert_block name="origin" />
       <axis xyz="0 1 0"/>
-      <limit lower="${-108.0/180.0 * pi}" upper="${128.25/180.0 * pi}" effort="0" velocity="0"/>
+      <limit lower="${-108.0/180.0 * pi}" upper="${128.25/180.0 * pi}" effort="10" velocity="1.0"/>
       <parent link="${parent}"/>
       <child link="${prefix}_uarm_joint"/>
@@ -114,8 +122,8 @@
       <axis xyz="1 0 0"/>
       <xacro:if value="${side=='right'}">
-        <limit lower="${-3.0375/180.0 * pi}" upper="${91.56375/180.0 * pi}" effort="0" velocity="0"/>
+        <limit lower="${-3.0375/180.0 * pi}" upper="${91.56375/180.0 * pi}" effort="10" velocity="1.0"/>
       </xacro:if>
       <xacro:if value="${side=='left'}">
-        <limit lower="${-91.56375/180.0 * pi}" upper="${3.0375/180.0 * pi}" effort="0" velocity="0"/>
+        <limit lower="${-91.56375/180.0 * pi}" upper="${3.0375/180.0 * pi}" effort="10" velocity="1.0"/>
       </xacro:if>
       <parent link="${prefix}_uarm_joint"/>
@@ -125,5 +133,5 @@
       <origin xyz="0.0088013 ${sign*0.060007} 0" rpy="0 0 0"/>
       <axis xyz="0 1 0"/>
-      <limit lower="${-128.68875/180.0 * pi}" upper="${134.325/180.0 * pi}" effort="0" velocity="0"/>
+      <limit lower="${-128.68875/180.0 * pi}" upper="${134.325/180.0 * pi}" effort="10" velocity="1.0"/>
       <parent link="${prefix}_uarm"/>
       <child link="${prefix}_larm_joint"/>
@@ -133,8 +141,8 @@
       <axis xyz="1 0 0"/>
       <xacro:if value="${side=='right'}">
-        <limit lower="${-13.5/180.0 * pi}" upper="${118.96875/180.0 * pi}" effort="0" velocity="0"/>
+        <limit lower="${-13.5/180.0 * pi}" upper="${118.96875/180.0 * pi}" effort="10" velocity="1.0"/>
       </xacro:if>
       <xacro:if value="${side=='left'}">
-        <limit lower="${-118.96875/180.0 * pi}" upper="${13.5/180.0 * pi}" effort="0" velocity="0"/>
+        <limit lower="${-118.96875/180.0 * pi}" upper="${13.5/180.0 * pi}" effort="10" velocity="1.0"/>
       </xacro:if>
       <parent link="${prefix}_larm_joint"/>
@@ -144,8 +152,13 @@
       <origin xyz="0 ${sign*0.061348} 0" rpy="0 0 0"/>
       <axis xyz="0 1 0"/>
-      <limit lower="${-135.0/180.0 * pi}" upper="${118.125/180.0 * pi}" effort="0" velocity="0"/>
+      <limit lower="${-135.0/180.0 * pi}" upper="${118.125/180.0 * pi}" effort="10" velocity="1.0"/>
       <parent link="${prefix}_larm"/>
       <child link="${prefix}_hand"/>
     </joint>
+    <joint name="${prefix}_hand_ee_fixed_joint" type="fixed">
+      <parent link="${prefix}_hand" />
+      <child link = "${prefix}_hand_ee" />
+      <origin xyz="0.0 0.0 0.0" rpy="0.0 0.0 0.0" />
+    </joint>
   </xacro:macro>
 </robot>

File: urdf/body.gazebo.xacro (robot description, xacro)
@@ -4,13 +4,30 @@
     <gazebo reference="body">
       <selfCollide>true</selfCollide>
+      <mu1>0.9</mu1>
+      <mu2>0.9</mu2>
     </gazebo>
     <gazebo reference="neck_pitch">
       <selfCollide>false</selfCollide>
+      <mu1>0.9</mu1>
+      <mu2>0.9</mu2>
     </gazebo>
     <gazebo reference="neck_yaw">
       <selfCollide>false</selfCollide>
+      <mu1>0.9</mu1>
+      <mu2>0.9</mu2>
     </gazebo>
     <gazebo reference="head">
-      <selfCollide>true</selfCollide>
+      <selfCollide>false</selfCollide>
+      <mu1>0.9</mu1>
+      <mu2>0.9</mu2>
+    </gazebo>
+    <gazebo reference="head_ny_joint">
+      <implicitSpringDamper>1</implicitSpringDamper>
+    </gazebo>
+    <gazebo reference="head_nz_joint">
+      <implicitSpringDamper>1</implicitSpringDamper>
+    </gazebo>
+    <gazebo reference="head_nx_joint">
+      <implicitSpringDamper>1</implicitSpringDamper>
     </gazebo>
   </xacro:macro>

File: urdf/body.urdf.xacro (robot description, xacro)
@@ -16,5 +16,5 @@
         <mass value="0.4426"/>
         <origin xyz="0.008509 0.000002 0.070698"/>
-        <inertia ixx="2871.143311e-10" ixy="-0.001151e-10" ixz="237.094467e-10" iyy="2672.078857e-10" iyz="-0.003379e-10" izz="1188.332153e-10"/>
+        <inertia ixx="2871.143311e-5" ixy="-0.001151e-5" ixz="237.094467e-5" iyy="2672.078857e-5" iyz="-0.003379e-5" izz="1188.332153e-5"/>
       </inertial>
     </link>
@@ -33,5 +33,5 @@
         <mass value="0.01"/>
         <origin xyz="-0.006449 0.000002 0.008964"/>
-        <inertia ixx="6.489763e-10" ixy="-0.000003e-10" ixz="-0.024047e-10" iyy="2.296302e-10" iyz="-0.000005e-10" izz="6.197822e-10"/>
+        <inertia ixx="6.489763e-5" ixy="-0.000003e-5" ixz="-0.024047e-5" iyy="2.296302e-5" iyz="-0.000005e-5" izz="6.197822e-5"/>
       </inertial>
     </link>
@@ -50,5 +50,5 @@
         <mass value="0.01"/>
         <origin xyz="0.008100 0.000002 0.017871"/>
-        <inertia ixx="12.636111e-10" ixy="-0.000001e-10" ixz="0.0" iyy="23.689224e-10" iyz="0.0" izz="17.372910e-10"/>
+        <inertia ixx="12.636111e-5" ixy="-0.000001e-5" ixz="0.0" iyy="23.689224e-5" iyz="0.0" izz="17.372910e-5"/>
       </inertial>
     </link>
@@ -67,5 +67,5 @@
         <mass value="0.1449"/>
         <origin xyz="0.014213 0.000001 0.011813"/>
-        <inertia ixx="650.041687e-10" ixy="-0.000280e-10" ixz="49.702934e-10" iyy="598.413635e-10" iyz="-0.000379e-10" izz="588.398682e-10"/>
+        <inertia ixx="650.041687e-5" ixy="-0.000280e-5" ixz="49.702934e-5" iyy="598.413635e-5" iyz="-0.000379e-5" izz="588.398682e-5"/>
       </inertial>
     </link>
@@ -78,5 +78,5 @@
       <origin xyz="0.0038738 0 0.132809" rpy="0 0 0"/>
       <axis xyz="0 1 0"/>
-      <limit lower="${-10.125/180.0 * pi}" upper="${23.625/180.0 * pi}" effort="0" velocity="0"/>
+      <limit lower="${-10.125/180.0 * pi}" upper="${23.625/180.0 * pi}" effort="10" velocity="1.0"/>
       <parent link="body"/>
       <child link="neck_pitch"/>
@@ -85,5 +85,5 @@
       <origin xyz="-0.0103485 0 0.011103" rpy="0 0 0"/>
       <axis xyz="0 0 1"/>
-      <limit lower="${-47.25/180.0 * pi}" upper="${47.25/180.0 * pi}" effort="0" velocity="0"/>
+      <limit lower="${-47.25/180.0 * pi}" upper="${47.25/180.0 * pi}" effort="10" velocity="1.0"/>
       <parent link="neck_pitch"/>
       <child link="head_yaw"/>
@@ -92,5 +92,5 @@
       <origin xyz="0 0 0.0129" rpy="0 0 0"/>
       <axis xyz="1 0 0"/>
-      <limit lower="${-21.9375/180.0 * pi}" upper="${28.6875/180.0 * pi}" effort="0" velocity="0"/>
+      <limit lower="${-21.9375/180.0 * pi}" upper="${28.6875/180.0 * pi}" effort="10" velocity="1.0"/>
       <parent link="head_yaw"/>
       <child link="head"/>

File: urdf/leg.gazebo.xacro (robot description, xacro)
@@ -3,20 +3,61 @@
   <xacro:macro name="premaidai_leg_gazebo" params="prefix">
     <gazebo reference="${prefix}_hip_joint">
-      <selfCollide>false</selfCollide>
+      <selfCollide>true</selfCollide>
+      <!-- <selfCollide>false</selfCollide> -->
+      <mu1>0.9</mu1>
+      <mu2>0.9</mu2>
     </gazebo>
     <gazebo reference="${prefix}_uleg_root">
-      <selfCollide>false</selfCollide>
+      <selfCollide>true</selfCollide>
+      <!-- <selfCollide>false</selfCollide> -->
+      <mu1>0.9</mu1>
+      <mu2>0.9</mu2>
     </gazebo>
     <gazebo reference="${prefix}_uleg">
-      <selfCollide>false</selfCollide>
+      <selfCollide>true</selfCollide>
+      <!-- <selfCollide>false</selfCollide> -->
+      <mu1>0.9</mu1>
+      <mu2>0.9</mu2>
     </gazebo>
     <gazebo reference="${prefix}_lleg">
-      <selfCollide>false</selfCollide>
+      <selfCollide>true</selfCollide>
+      <!-- <selfCollide>false</selfCollide> -->
+      <mu1>0.9</mu1>
+      <mu2>0.9</mu2>
     </gazebo>
     <gazebo reference="${prefix}_ankle">
-      <selfCollide>false</selfCollide>
+      <selfCollide>true</selfCollide>
+      <!-- <selfCollide>false</selfCollide> -->
+      <mu1>0.9</mu1>
+      <mu2>0.9</mu2>
     </gazebo>
     <gazebo reference="${prefix}_foot">
-      <selfCollide>false</selfCollide>
+      <selfCollide>true</selfCollide>
+      <!-- <selfCollide>false</selfCollide> -->
+      <kp>1000000.0</kp>
+      <kd>100.0</kd>
+      <mu1>1.5</mu1>
+      <mu2>1.5</mu2>
+      <fdir1>1 0 0</fdir1>
+      <maxVel>1.0</maxVel>
+      <minDepth>0.00</minDepth>
+    </gazebo>
+    <gazebo reference="${prefix}_hpz_joint">
+      <implicitSpringDamper>1</implicitSpringDamper>
+    </gazebo>
+    <gazebo reference="${prefix}_hpx_joint">
+      <implicitSpringDamper>1</implicitSpringDamper>
+    </gazebo>
+    <gazebo reference="${prefix}_hpy_joint">
+      <implicitSpringDamper>1</implicitSpringDamper>
+    </gazebo>
+    <gazebo reference="${prefix}_kny_joint">
+      <implicitSpringDamper>1</implicitSpringDamper>
+    </gazebo>
+    <gazebo reference="${prefix}_aky_joint">
+      <implicitSpringDamper>1</implicitSpringDamper>
+    </gazebo>
+    <gazebo reference="${prefix}_akx_joint">
+      <implicitSpringDamper>1</implicitSpringDamper>
     </gazebo>
   </xacro:macro>

File: urdf/leg.urdf.xacro (robot description, xacro)
@@ -24,5 +24,5 @@
         <mass value="0.0143"/>
         <origin xyz="0.000000 ${sign*0.000183} -0.010532"/>
-        <inertia ixx="20.138887e-10" ixy="-0.000001e-10" ixz="0.0e-10" iyy="53.757824e-10" iyz="${sign*-0.518773e-10}" izz="46.127151e-10"/>
+        <inertia ixx="20.138887e-5" ixy="-0.000001e-5" ixz="0.0e-5" iyy="53.757824e-5" iyz="${sign*-0.518773e-5}" izz="46.127151e-5"/>
       </inertial>
     </link>
@@ -43,5 +43,5 @@
         <mass value="0.0648"/>
         <origin xyz="-0.000000 ${sign*0.013420} -0.004373"/>
-        <inertia ixx="246.003845e-10" ixy="${sign*-0.001517e-10}" ixz="-0.001688e-10" iyy="191.922195e-10" iyz="${sign*-6.165664e-10}" izz="238.454895e-10"/>
+        <inertia ixx="246.003845e-5" ixy="${sign*-0.001517e-5}" ixz="-0.001688e-5" iyy="191.922195e-5" iyz="${sign*-6.165664e-5}" izz="238.454895e-5"/>
       </inertial>
     </link>
@@ -62,5 +62,5 @@
         <mass value="0.1134"/>
         <origin xyz="-0.000000 0.000001 -0.032601"/>
-        <inertia ixx="884.390869e-10" ixy="0.000002e-10" ixz="-0.000046e-10" iyy="825.489990e-10" iyz="-0.000031e-10" izz="222.801773e-10"/>
+        <inertia ixx="884.390869e-5" ixy="0.000002e-5" ixz="-0.000046e-5" iyy="825.489990e-5" iyz="-0.000031e-5" izz="222.801773e-5"/>
       </inertial>
     </link>
@@ -81,5 +81,5 @@
         <mass value="0.0719"/>
         <origin xyz="-0.001624 ${sign*0.002494} -0.034776"/>
-        <inertia ixx="735.568420e-10" ixy="${sign*-1.871153e-10}" ixz="-35.647034e-10" iyy="434.662354e-10" iyz="${sign*0.247592e-10}" izz="480.555054e-10"/>
+        <inertia ixx="735.568420e-5" ixy="${sign*-1.871153e-5}" ixz="-35.647034e-5" iyy="434.662354e-5" iyz="${sign*0.247592e-5}" izz="480.555054e-5"/>
       </inertial>
     </link>
@@ -100,5 +100,5 @@
         <mass value="0.0571"/>
         <origin xyz="-0.009629 0.000379 -0.003702"/>
-        <inertia ixx="175.244446e-10" ixy="-0.000004e-10" ixz="11.289989e-10" iyy="257.425598e-10" iyz="-0.000002e-10" izz="224.547821e-10"/>
+        <inertia ixx="175.244446e-5" ixy="-0.000004e-5" ixz="11.289989e-5" iyy="257.425598e-5" iyz="-0.000002e-5" izz="224.547821e-5"/>
       </inertial>
     </link>
@@ -119,5 +119,5 @@
         <mass value="0.0941"/>
         <origin xyz="0.005014 ${sign*0.008793} -0.004123"/>
-        <inertia ixx="383.406982e-10" ixy="${sign*11.222215e-10}" ixz="12.157411e-10" iyy="1013.430359e-10" iyz="${sign*-1.649494e-10}" izz="1206.411377e-10"/>
+        <inertia ixx="383.406982e-5" ixy="${sign*11.222215e-5}" ixz="12.157411e-5" iyy="1013.430359e-5" iyz="${sign*-1.649494e-5}" izz="1206.411377e-5"/>
       </inertial>
     </link>
@@ -125,5 +125,5 @@
       <xacro:insert_block name="origin" />
       <axis xyz="0 0 1"/>
-      <limit lower="${-81.0/180.0 * pi}" upper="${102.43/180.0 * pi}" effort="0" velocity="0"/>
+      <limit lower="${-81.0/180.0 * pi}" upper="${102.43/180.0 * pi}" effort="10" velocity="1.0"/>
       <parent link="${parent}"/>
       <child link="${prefix}_hip_joint"/>
@@ -133,8 +133,8 @@
       <axis xyz="1 0 0"/>
       <xacro:if value="${side=='right'}">
-        <limit lower="${-25.35/180.0 * pi}" upper="${22.713/180.0 * pi}" effort="0" velocity="0"/>
+        <limit lower="${-25.35/180.0 * pi}" upper="${22.713/180.0 * pi}" effort="10" velocity="1.0"/>
       </xacro:if>
       <xacro:if value="${side=='left'}">
-        <limit lower="${-22.713/180.0 * pi}" upper="${25.35/180.0 * pi}" effort="0" velocity="0"/>
+        <limit lower="${-22.713/180.0 * pi}" upper="${25.35/180.0 * pi}" effort="10" velocity="1.0"/>
       </xacro:if>
       <parent link="${prefix}_hip_joint"/>
@@ -144,5 +144,5 @@
       <origin xyz="0 ${sign*0.0128525} -0.034358" rpy="0 0 0"/>
       <axis xyz="0 1 0"/>
-      <limit lower="${-91.60/180.0 * pi}" upper="${90.213/180.0 * pi}" effort="0" velocity="0"/>
+      <limit lower="${-91.60/180.0 * pi}" upper="${90.213/180.0 * pi}" effort="10" velocity="1.0"/>
       <parent link="${prefix}_uleg_root"/>
       <child link="${prefix}_uleg"/>
@@ -151,5 +151,5 @@
       <origin xyz="0 0 -0.0652" rpy="0 0 0"/>
       <axis xyz="0 1 0"/>
-      <limit lower="${-2.0925/180.0 * pi}" upper="${119.64/180.0 * pi}" effort="0" velocity="0"/>
+      <limit lower="${-2.0925/180.0 * pi}" upper="${119.64/180.0 * pi}" effort="10" velocity="1.0"/>
       <parent link="${prefix}_uleg"/>
       <child link="${prefix}_lleg"/>
@@ -158,5 +158,5 @@
       <origin xyz="0 0 -0.065" rpy="0 0 0"/>
       <axis xyz="0 1 0"/>
-      <limit lower="${-61.3575/180.0 * pi}" upper="${24.3/180.0 * pi}" effort="0" velocity="0"/>
+      <limit lower="${-61.3575/180.0 * pi}" upper="${24.3/180.0 * pi}" effort="10" velocity="1.0"/>
       <parent link="${prefix}_lleg"/>
       <child link="${prefix}_ankle"/>
@@ -166,8 +166,8 @@
       <axis xyz="1 0 0"/>
       <xacro:if value="${side=='right'}">
-        <limit lower="${-38.23875/180.0 * pi}" upper="${37.29375/180.0 * pi}" effort="0" velocity="0"/>
+        <limit lower="${-38.23875/180.0 * pi}" upper="${37.29375/180.0 * pi}" effort="10" velocity="1.0"/>
       </xacro:if>
       <xacro:if value="${side=='left'}">
-        <limit lower="${-37.29375/180.0 * pi}" upper="${38.23875/180.0 * pi}" effort="0" velocity="0"/>
+        <limit lower="${-37.29375/180.0 * pi}" upper="${38.23875/180.0 * pi}" effort="10" velocity="1.0"/>
       </xacro:if>
       <parent link="${prefix}_ankle"/>
